Commit message: Added transmissions for fingers; fixed gazebo link names; only one gazebo_ros_control.

File: victor_description/urdf/dual_iiwa7_no_torso.xacro (robot description, xacro)
@@ -5,5 +5,5 @@
   <!--Import the lbr iiwa macro -->
   <xacro:include filename="$(find victor_description)/urdf/iiwa7.xacro"/>
-  <xacro:arg name="hardware_interface" default="PositionJointInterface"/>
+  <xacro:arg name="hardware_interface" default="hardware_interface/PositionJointInterface"/>
   <!--<xacro:arg name="robot_name" default="iiwa"/>-->
   <!-- Fix to world just for testing -->

File: victor_description/urdf/iiwa.gazebo.xacro (robot description, xacro)
@@ -3,11 +3,13 @@
   <xacro:macro name="iiwa_gazebo" params="robot_name">
     <!-- Load Gazebo lib and set the robot namespace -->
-    <gazebo>
-      <plugin name="gazebo_ros_control" filename="libgazebo_ros_control.so">
-        <robotNamespace>/${robot_name}</robotNamespace>
-      </plugin>
-    </gazebo>
+    <!--<xacro:if value="${load_control_plugin}">-->
+      <!--<gazebo>-->
+        <!--<plugin name="gazebo_ros_control" filename="libgazebo_ros_control.so">-->
+          <!--<robotNamespace>/${robot_name}</robotNamespace>-->
+        <!--</plugin>-->
+      <!--</gazebo>-->
+    <!--</xacro:if>-->
     <!-- Link0 -->
-    <gazebo reference="iiwa_link_0">
+    <gazebo reference="${robot_name}_link_0">
       <material>Gazebo/Grey</material>
       <mu1>0.2</mu1>
@@ -15,5 +17,5 @@
     </gazebo>
     <!-- Link1 -->
-    <gazebo reference="iiwa_link_1">
+    <gazebo reference="${robot_name}_link_1">
       <material>Gazebo/Orange</material>
       <mu1>0.2</mu1>
@@ -21,5 +23,5 @@
     </gazebo>
     <!-- Link2 -->
-    <gazebo reference="iiwa_link_2">
+    <gazebo reference="${robot_name}_link_2">
       <material>Gazebo/Orange</material>
       <mu1>0.2</mu1>
@@ -27,5 +29,5 @@
     </gazebo>
     <!-- Link3 -->
-    <gazebo reference="iiwa_link_3">
+    <gazebo reference="${robot_name}_link_3">
       <material>Gazebo/Orange</material>
       <mu1>0.2</mu1>
@@ -33,5 +35,5 @@
     </gazebo>
     <!-- Link4 -->
-    <gazebo reference="iiwa_link_4">
+    <gazebo reference="${robot_name}_link_4">
       <material>Gazebo/Orange</material>
       <mu1>0.2</mu1>
@@ -39,5 +41,5 @@
     </gazebo>
     <!-- Link5 -->
-    <gazebo reference="iiwa_link_5">
+    <gazebo reference="${robot_name}_link_5">
       <material>Gazebo/Orange</material>
       <mu1>0.2</mu1>
@@ -45,5 +47,5 @@
     </gazebo>
     <!-- Link6 -->
-    <gazebo reference="iiwa_link_6">
+    <gazebo reference="${robot_name}_link_6">
       <material>Gazebo/Orange</material>
       <mu1>0.2</mu1>
@@ -51,5 +53,5 @@
     </gazebo>
     <!-- Link7 -->
-    <gazebo reference="iiwa_link_7">
+    <gazebo reference="${robot_name}_link_7">
       <material>Gazebo/Grey</material>
       <mu1>0.2</mu1>

File: victor_description/urdf/iiwa.transmission.xacro (robot description, xacro)
@@ -1,80 +1,66 @@
 <?xml version="1.0"?>
 <robot xmlns:xacro="http://www.ros.org/wiki/xacro">
-  <xacro:macro name="iiwa_transmission" params="hardware_interface">
-    <transmission name="iiwa_tran_1">
-      <robotNamespace>/${robot_name}</robotNamespace>
+  <xacro:macro name="iiwa_transmission" params="hardware_interface robot_name">
+    <transmission name="${robot_name}_tran_1">
       <type>transmission_interface/SimpleTransmission</type>
-      <joint name="iiwa_joint_1">
-	<hardwareInterface>${hardware_interface}</hardwareInterface>
+      <joint name="${robot_name}_joint_1">
+        <hardwareInterface>${hardware_interface}</hardwareInterface>
       </joint>
-      <actuator name="iiwa_motor_1">
-	<hardwareInterface>${hardware_interface}</hardwareInterface>
-	<mechanicalReduction>1</mechanicalReduction>
+      <actuator name="${robot_name}_motor_1">
+        <mechanicalReduction>1</mechanicalReduction>
       </actuator>
     </transmission>
-    <transmission name="iiwa_tran_2">
-      <robotNamespace>/${robot_name}</robotNamespace>
+    <transmission name="${robot_name}_tran_2">
       <type>transmission_interface/SimpleTransmission</type>
-      <joint name="iiwa_joint_2">
-	<hardwareInterface>${hardware_interface}</hardwareInterface>
+      <joint name="${robot_name}_joint_2">
+        <hardwareInterface>${hardware_interface}</hardwareInterface>
       </joint>
-      <actuator name="iiwa_motor_2">
-	<hardwareInterface>${hardware_interface}</hardwareInterface>
-	<mechanicalReduction>1</mechanicalReduction>
+      <actuator name="${robot_name}_motor_2">
+        <mechanicalReduction>1</mechanicalReduction>
       </actuator>
     </transmission>
-    <transmission name="iiwa_tran_3">
-      <robotNamespace>/${robot_name}</robotNamespace>
+    <transmission name="${robot_name}_tran_3">
       <type>transmission_interface/SimpleTransmission</type>
-      <joint name="iiwa_joint_3">
-	<hardwareInterface>${hardware_interface}</hardwareInterface>
+      <joint name="${robot_name}_joint_3">
+        <hardwareInterface>${hardware_interface}</hardwareInterface>
       </joint>
-      <actuator name="iiwa_motor_3">
-	<hardwareInterface>${hardware_interface}</hardwareInterface>
-	<mechanicalReduction>1</mechanicalReduction>
+      <actuator name="${robot_name}_motor_3">
+        <mechanicalReduction>1</mechanicalReduction>
       </actuator>
     </transmission>
-    <transmission name="iiwa_tran_4">
-      <robotNamespace>/${robot_name}</robotNamespace>
+    <transmission name="${robot_name}_tran_4">
       <type>transmission_interface/SimpleTransmission</type>
-      <joint name="iiwa_joint_4">
-	<hardwareInterface>${hardware_interface}</hardwareInterface>
+      <joint name="${robot_name}_joint_4">
+        <hardwareInterface>${hardware_interface}</hardwareInterface>
       </joint>
-      <actuator name="iiwa_motor_4">
-	<hardwareInterface>${hardware_interface}</hardwareInterface>
-	<mechanicalReduction>1</mechanicalReduction>
+      <actuator name="${robot_name}_motor_4">
+        <mechanicalReduction>1</mechanicalReduction>
       </actuator>
     </transmission>
-    <transmission name="iiwa_tran_5">
-      <robotNamespace>/${robot_name}</robotNamespace>
+    <transmission name="${robot_name}_tran_5">
       <type>transmission_interface/SimpleTransmission</type>
-      <joint name="iiwa_joint_5">
-	<hardwareInterface>${hardware_interface}</hardwareInterface>
+      <joint name="${robot_name}_joint_5">
+        <hardwareInterface>${hardware_interface}</hardwareInterface>
       </joint>
-      <actuator name="iiwa_motor_5">
-	<hardwareInterface>${hardware_interface}</hardwareInterface>
-	<mechanicalReduction>1</mechanicalReduction>
+      <actuator name="${robot_name}_motor_5">
+        <mechanicalReduction>1</mechanicalReduction>
       </actuator>
     </transmission>
-    <transmission name="iiwa_tran_6">
-      <robotNamespace>/${robot_name}</robotNamespace>
+    <transmission name="${robot_name}_tran_6">
       <type>transmission_interface/SimpleTransmission</type>
-      <joint name="iiwa_joint_6">
-	<hardwareInterface>${hardware_interface}</hardwareInterface>
+      <joint name="${robot_name}_joint_6">
+        <hardwareInterface>${hardware_interface}</hardwareInterface>
       </joint>
-      <actuator name="iiwa_motor_6">
-	<hardwareInterface>${hardware_interface}</hardwareInterface>
-	<mechanicalReduction>1</mechanicalReduction>
+      <actuator name="${robot_name}_motor_6">
+        <mechanicalReduction>1</mechanicalReduction>
       </actuator>
     </transmission>
-    <transmission name="iiwa_tran_7">
-      <robotNamespace>/${robot_name}</robotNamespace>
+    <transmission name="${robot_name}_tran_7">
       <type>transmission_interface/SimpleTransmission</type>
-      <joint name="iiwa_joint_7">
-	<hardwareInterface>${hardware_interface}</hardwareInterface>
+      <joint name="${robot_name}_joint_7">
+        <hardwareInterface>${hardware_interface}</hardwareInterface>
       </joint>
-      <actuator name="iiwa_motor_7">
-	<hardwareInterface>${hardware_interface}</hardwareInterface>
-	<mechanicalReduction>1</mechanicalReduction>
+      <actuator name="${robot_name}_motor_7">
+        <mechanicalReduction>1</mechanicalReduction>
       </actuator>
     </transmission>

File: victor_description/urdf/iiwa7.xacro (robot description, xacro)
@@ -9,5 +9,5 @@
     <!-- some constants -->
     <xacro:property name="safety_controller_k_pos" value="100"/>
-    <xacro:property name="safety_controller_k_vel" value="2"/>
+    <xacro:property name="safety_controller_k_vel" value="100"/>
     <xacro:property name="joint_damping" value="0.5"/>
     <xacro:property name="max_effort" value="300"/>
@@ -303,5 +303,6 @@
         <!--Extensions -->
         <xacro:iiwa_gazebo robot_name="${robot_name}"/>
-        <xacro:iiwa_transmission hardware_interface="${hardware_interface}"/>
+        <xacro:iiwa_transmission hardware_interface="${hardware_interface}"
+                                 robot_name="${robot_name}"/>
     </xacro:macro>
 </robot>

File: victor_description/urdf/robotiq_3finger_gripper.xacro (robot description, xacro)
@@ -2,5 +2,6 @@
 <robot xmlns:xacro="http://www.ros.org/wiki/xacro">
     <xacro:include filename="$(find victor_description)/urdf/robotiq_finger.xacro"/>
-    <xacro:macro name="robotiq_3finger" params="parent prefix *origin">
+    <xacro:include filename="$(find victor_description)/urdf/robotiq_3finger_gripper.transmission.xacro"/>
+    <xacro:macro name="robotiq_3finger" params="parent prefix hardware_interface *origin">
         <joint name="${prefix}_palm_joint" type="fixed">
             <xacro:insert_block name="origin"/>
@@ -82,4 +83,6 @@
         </joint>
         <xacro:robotiq_finger prefix="${prefix}_fingerC"/>
+        <xacro:robotiq_3finger_gripper_transmission hardware_interface="${hardware_interface}"
+                                                    robot_name="${prefix}"/>
     </xacro:macro>
 </robot>

File: victor_description/urdf/robotiq_finger.xacro (robot description, xacro)
@@ -2,5 +2,5 @@
 <robot xmlns:xacro="http://www.ros.org/wiki/xacro">
     <xacro:property name="safety_controller_k_pos" value="100"/>
-    <xacro:property name="safety_controller_k_vel" value="2"/>
+    <xacro:property name="safety_controller_k_vel" value="100"/>
     <xacro:property name="joint_damping" value="0.5"/>
     <xacro:property name="max_effort" value="300"/>

File: victor_description/urdf/victor.urdf.xacro (robot description, xacro)
@@ -2,5 +2,5 @@
 <robot name="victor" xmlns:xacro="http://www.ros.org/wiki/xacro">
     <xacro:arg name="robot_name" default="victor"/>
-    <xacro:arg name="hardware_interface" default="PositionJointInterface"/>
+    <xacro:arg name="hardware_interface" default="hardware_interface/PositionJointInterface"/>
     <!-- Import Rviz colors -->
     <xacro:include filename="$(find victor_description)/urdf/materials.xacro"/>
@@ -47,8 +47,8 @@
     <!--Import the Robotiq 3 finger macro -->
     <xacro:include filename="$(find victor_description)/urdf/robotiq_3finger_gripper.xacro"/>
-    <xacro:robotiq_3finger parent="$(arg robot_name)_left_gripper_mounting_bracket" prefix="$(arg robot_name)_left_gripper">
+    <xacro:robotiq_3finger parent="$(arg robot_name)_left_gripper_mounting_bracket" prefix="$(arg robot_name)_left_gripper" hardware_interface="$(arg hardware_interface)">
         <origin xyz="0 0 0.02705" rpy="0 0 ${PI/4}"/> <!-- Offset measured with a tape measure; please confirm/fix this value -->
     </xacro:robotiq_3finger>
-    <xacro:robotiq_3finger parent="$(arg robot_name)_right_gripper_mounting_bracket" prefix="$(arg robot_name)_right_gripper">
+    <xacro:robotiq_3finger parent="$(arg robot_name)_right_gripper_mounting_bracket" prefix="$(arg robot_name)_right_gripper" hardware_interface="$(arg hardware_interface)">
         <origin xyz="0 0 0.02705" rpy="0 0 ${PI/4}"/> <!-- Offset measured with a tape measure; please confirm/fix this value -->
     </xacro:robotiq_3finger>
@@ -56,3 +56,9 @@
     <xacro:include filename="$(find victor_description)/urdf/robotiq_pinch_grasp_tools.xacro"/>
     <xacro:robotiq_pinch_grasp_tools robot_name="$(arg robot_name)"/>
+    <!-- Add Gazebo properties for whole robot -->
+    <xacro:include filename="$(find victor_description)/urdf/gazebo_utilities.xacro"/>
+    <!-- Load Gazebo lib and set the robot namespace -->
+    <xacro:add_gazebo_control_plugin robot_namespace="$(arg robot_name)"/>
+    <!-- Rigidly attach Victor to the Gazebo world -->
+    <xacro:add_gazebo_fixed_link base_link="$(arg robot_name)_root"/>
 </robot>
