Commit message: Cleaning up utilities.

File: victor_description/urdf/utilities.xacro (robot description, xacro)
@@ -6,14 +6,14 @@
   <!--Cuboid-->
   <xacro:macro name="cuboid_inertia" params="width height length mass">
-    <inertia ixx="${mass * (height * height + length * length) / 12)}"
-             iyy="${mass * (width * width + length * length) / 12)}"
-             izz="${mass * (width * width + height * height) / 12)}"
+    <inertia ixx="${mass * (height * height + length * length) / 12}"
+             iyy="${mass * (width * width + length * length) / 12}"
+             izz="${mass * (width * width + height * height) / 12}"
              ixy="0" iyz="0" ixz="0"/>
   </xacro:macro>
   <!--Cylinder: length is along the y-axis! -->
   <xacro:macro name="cylinder_inertia" params="radius length mass">
-    <inertia ixx="${mass * (3 * radius * radius + length * length) / 12)}"
-             iyy="${mass * radius* radius / 2)}"
-             izz="${mass * (3 * radius * radius + length * length) / 12)}"
+    <inertia ixx="${mass * (3 * radius * radius + length * length) / 12}"
+             iyy="${mass * radius* radius / 2}"
+             izz="${mass * (3 * radius * radius + length * length) / 12}"
              ixy="0" iyz="0" ixz="0"/>
   </xacro:macro>

File: victor_description/urdf/victor.urdf.xacro (robot description, xacro)
@@ -61,4 +61,6 @@
     <xacro:add_gazebo_control_plugin robot_namespace="$(arg robot_name)"/>
     <!-- Rigidly attach Victor to the Gazebo world -->
+    <!--
     <xacro:add_gazebo_fixed_link base_link="$(arg robot_name)_root"/>
+    -->
 </robot>
