Commit message: rework of gazebo simulation
squash of peter branch

File: victor_description/urdf/iiwa7.xacro (robot description, xacro)
@@ -9,6 +9,6 @@
     <!-- some constants -->
     <xacro:property name="safety_controller_k_pos" value="100"/>
-    <xacro:property name="safety_controller_k_vel" value="2"/>
-    <xacro:property name="joint_damping" value="0.5"/>
+    <xacro:property name="safety_controller_k_vel" value="100"/>
+    <xacro:property name="joint_damping" value="0.2"/>
     <xacro:property name="max_effort" value="300"/>
     <xacro:property name="max_velocity" value="10"/>
@@ -303,5 +303,6 @@
         <!--Extensions -->
         <xacro:iiwa_gazebo robot_name="${robot_name}"/>
-        <xacro:iiwa_transmission hardware_interface="${hardware_interface}"/>
+        <xacro:iiwa_transmission hardware_interface="${hardware_interface}"
+                                 robot_name="${robot_name}"/>
     </xacro:macro>
 </robot>

File: victor_description/urdf/robotiq_3finger_gripper.xacro (robot description, xacro)
@@ -2,5 +2,7 @@
 <robot xmlns:xacro="http://www.ros.org/wiki/xacro">
     <xacro:include filename="$(find victor_description)/urdf/robotiq_finger.xacro"/>
-    <xacro:macro name="robotiq_3finger" params="parent prefix *origin">
+    <xacro:include filename="$(find victor_description)/urdf/robotiq_3finger_gripper.transmission.xacro"/>
+    <xacro:macro name="robotiq_3finger" params="parent prefix hardware_interface *origin">
+        <xacro:property name="joint_damping" value="0.05"/>
         <joint name="${prefix}_palm_joint" type="fixed">
             <xacro:insert_block name="origin"/>
@@ -51,5 +53,5 @@
             <child link="${prefix}_fingerA_base"/>
         </joint>
-        <xacro:robotiq_finger prefix="${prefix}_fingerA"/>
+        <xacro:robotiq_finger prefix="${prefix}_fingerA" joint_damping="${joint_damping}"/>
         <!-- Finger B -->
         <joint name="${prefix}_fingerB_knuckle" type="revolute">
@@ -60,11 +62,7 @@
             <limit lower="${-16 * PI / 180}" upper="${10 * PI / 180}"
                effort="${max_effort}" velocity="${max_velocity}"/>
-            <safety_controller soft_lower_limit="${-14 * PI / 180}"
-                               soft_upper_limit="${8 * PI / 180}"
-                               k_position="${safety_controller_k_pos}"
-                               k_velocity="${safety_controller_k_vel}"/>
             <dynamics damping="${joint_damping}"/>
         </joint>
-        <xacro:robotiq_finger prefix="${prefix}_fingerB"/>
+        <xacro:robotiq_finger prefix="${prefix}_fingerB" joint_damping="${joint_damping}"/>
         <!-- Finger C -->
         <joint name="${prefix}_fingerC_knuckle" type="revolute">
@@ -75,11 +73,9 @@
             <limit lower="${-16 * PI / 180}" upper="${10 * PI / 180}"
                effort="${max_effort}" velocity="${max_velocity}"/>
-            <safety_controller soft_lower_limit="${-14 * PI / 180}"
-                               soft_upper_limit="${8 * PI / 180}"
-                               k_position="${safety_controller_k_pos}"
-                               k_velocity="${safety_controller_k_vel}"/>
             <dynamics damping="${joint_damping}"/>
         </joint>
-        <xacro:robotiq_finger prefix="${prefix}_fingerC"/>
+        <xacro:robotiq_finger prefix="${prefix}_fingerC" joint_damping="${joint_damping}"/>
+        <xacro:robotiq_3finger_gripper_transmission hardware_interface="${hardware_interface}"
+                                                    robot_name="${prefix}"/>
     </xacro:macro>
 </robot>

File: victor_description/urdf/robotiq_finger.xacro (robot description, xacro)
@@ -1,15 +1,12 @@
 <?xml version="1.0"?>
 <robot xmlns:xacro="http://www.ros.org/wiki/xacro">
-    <xacro:property name="safety_controller_k_pos" value="100"/>
-    <xacro:property name="safety_controller_k_vel" value="2"/>
-    <xacro:property name="joint_damping" value="0.5"/>
     <xacro:property name="max_effort" value="300"/>
     <xacro:property name="max_velocity" value="10"/>
-    <xacro:macro name="robotiq_finger" params="prefix">
+    <xacro:macro name="robotiq_finger" params="prefix joint_damping">
         <link name="${prefix}_base">
             <inertial>
                 <origin xyz="0 0 0" rpy="0 0 0"/>
-                <mass value="1"/>
-                <inertia ixx="0.01" ixy="0" ixz="0" iyy="0.01" iyz="0" izz="0.01"/>
+                <mass value="0.1"/>
+                <inertia ixx="0.0001667" ixy="0" ixz="0" iyy="0.0001667" iyz="0" izz="0.0001667"/>
             </inertial>
             <visual>
@@ -36,8 +33,4 @@
             <limit lower="0" upper="1.2217304763960307"
                    effort="${max_effort}" velocity="${max_velocity}"/>
-            <safety_controller soft_lower_limit="${-35 * PI / 180}"
-                               soft_upper_limit="${35 * PI / 180}"
-                               k_position="${safety_controller_k_pos}"
-                               k_velocity="${safety_controller_k_vel}"/>
             <dynamics damping="${joint_damping}"/>
         </joint>
@@ -45,6 +38,6 @@
             <inertial>
                 <origin xyz="0 0 0" rpy="0 0 0"/>
-                <mass value="1"/>
-                <inertia ixx="0.01" ixy="0" ixz="0" iyy="0.01" iyz="0" izz="0.01"/>
+                <mass value="0.1"/>
+                <inertia ixx="0.0001667" ixy="0" ixz="0" iyy="0.0001667" iyz="0" izz="0.0001667"/>
             </inertial>
             <visual>
@@ -71,8 +64,4 @@
             <limit lower="-1" upper="1"
                    effort="${max_effort}" velocity="${max_velocity}"/>
-            <safety_controller soft_lower_limit="${0 * PI / 180}"
-                               soft_upper_limit="${90 * PI / 180}"
-                               k_position="${safety_controller_k_pos}"
-                               k_velocity="${safety_controller_k_vel}"/>
             <dynamics damping="${joint_damping}"/>
         </joint>
@@ -80,6 +69,6 @@
             <inertial>
                 <origin xyz="0 0 0" rpy="0 0 0"/>
-                <mass value="1"/>
-                <inertia ixx="0.01" ixy="0" ixz="0" iyy="0.01" iyz="0" izz="0.01"/>
+                <mass value="0.1"/>
+                <inertia ixx="0.0001667" ixy="0" ixz="0" iyy="0.0001667" iyz="0" izz="0.0001667"/>
             </inertial>
             <visual>
@@ -106,8 +95,4 @@
             <limit lower="-1" upper="1"
                    effort="${max_effort}" velocity="${max_velocity}"/>
-            <safety_controller soft_lower_limit="${-25 * PI / 180}"
-                               soft_upper_limit="${73 * PI / 180}"
-                               k_position="${safety_controller_k_pos}"
-                               k_velocity="${safety_controller_k_vel}"/>
             <dynamics damping="${joint_damping}"/>
         </joint>
@@ -115,6 +100,6 @@
             <inertial>
                 <origin xyz="0 0 0" rpy="0 0 0"/>
-                <mass value="1"/>
-                <inertia ixx="0.01" ixy="0" ixz="0" iyy="0.01" iyz="0" izz="0.01"/>
+                <mass value="0.1"/>
+                <inertia ixx="0.0001667" ixy="0" ixz="0" iyy="0.0001667" iyz="0" izz="0.0001667"/>
             </inertial>
             <visual>

File: victor_description/urdf/victor.urdf.xacro (robot description, xacro)
@@ -2,5 +2,5 @@
 <robot name="victor" xmlns:xacro="http://www.ros.org/wiki/xacro">
     <xacro:arg name="robot_name" default="victor"/>
-    <xacro:arg name="hardware_interface" default="PositionJointInterface"/>
+    <xacro:arg name="hardware_interface" default="hardware_interface/EffortJointInterface"/>
     <!-- Import Rviz colors -->
     <xacro:include filename="$(find victor_description)/urdf/materials.xacro"/>
@@ -47,8 +47,10 @@
     <!--Import the Robotiq 3 finger macro -->
     <xacro:include filename="$(find victor_description)/urdf/robotiq_3finger_gripper.xacro"/>
-    <xacro:robotiq_3finger parent="$(arg robot_name)_left_gripper_mounting_bracket" prefix="$(arg robot_name)_left_gripper">
+    <xacro:robotiq_3finger parent="$(arg robot_name)_left_gripper_mounting_bracket" prefix="$(arg robot_name)_left_gripper"
+                           hardware_interface="$(arg hardware_interface)">
         <origin xyz="0 0 0.02705" rpy="0 0 ${PI/4}"/> <!-- Offset measured with a tape measure; please confirm/fix this value -->
     </xacro:robotiq_3finger>
-    <xacro:robotiq_3finger parent="$(arg robot_name)_right_gripper_mounting_bracket" prefix="$(arg robot_name)_right_gripper">
+    <xacro:robotiq_3finger parent="$(arg robot_name)_right_gripper_mounting_bracket" prefix="$(arg robot_name)_right_gripper"
+                           hardware_interface="$(arg hardware_interface)">
         <origin xyz="0 0 0.02705" rpy="0 0 ${PI/4}"/> <!-- Offset measured with a tape measure; please confirm/fix this value -->
     </xacro:robotiq_3finger>
@@ -56,3 +58,13 @@
     <xacro:include filename="$(find victor_description)/urdf/robotiq_pinch_grasp_tools.xacro"/>
     <xacro:robotiq_pinch_grasp_tools robot_name="$(arg robot_name)"/>
+    <!-- Add Gazebo properties for whole robot -->
+    <xacro:include filename="$(find victor_description)/urdf/victor.gazebo.xacro"/>
+    <xacro:include filename="$(find victor_description)/urdf/gazebo_utilities.xacro"/>
+    <!-- Load Gazebo lib and set the robot namespace -->
+    <xacro:add_gazebo_control_plugin robot_namespace="$(arg robot_name)"/>
+    <xacro:add_moveit_planning_scene_plugin robot_namespace="$(arg robot_name)" root_frame_id="victor_root"/>
+    <xacro:add_simulation_compliance side="left"/>
+    <xacro:add_simulation_compliance side="right"/>
+    <!-- Rigidly attach Victor to the Gazebo world -->
+    <xacro:add_gazebo_fixed_link base_link="$(arg robot_name)_root"/>
 </robot>

Commit message: ignore all gripper collisions in planning

File: victor_description/urdf/iiwa7.xacro (robot description, xacro)
@@ -10,5 +10,5 @@
     <xacro:property name="safety_controller_k_pos" value="100"/>
     <xacro:property name="safety_controller_k_vel" value="100"/>
-    <xacro:property name="joint_damping" value="0.5"/>
+    <xacro:property name="joint_damping" value="0.2"/>
     <xacro:property name="max_effort" value="300"/>
     <xacro:property name="max_velocity" value="10"/>
