Commit message: de-duplicate transmissions

File: victor_description/urdf/robotiq_3finger_gripper.transmission.xacro (robot description, xacro)
@@ -2,83 +2,83 @@
 <robot xmlns:xacro="http://www.ros.org/wiki/xacro">
     <xacro:include filename="$(find victor_description)/urdf/gazebo_utilities.xacro"/>
-    <xacro:macro name="robotiq_transmissions" params="hardware_interface">
-        <xacro:add_transmission joint_name="l_palm_finger_1_joint" hardware_interface="${hardware_interface}"/>
-        <xacro:add_transmission joint_name="l_finger_1_joint_1" hardware_interface="${hardware_interface}"/>
-        <xacro:add_transmission joint_name="l_finger_1_joint_2" hardware_interface="${hardware_interface}"/>
-        <xacro:add_transmission joint_name="l_finger_1_joint_3" hardware_interface="${hardware_interface}"/>
-        <xacro:add_transmission joint_name="l_palm_finger_2_joint" hardware_interface="${hardware_interface}"/>
-        <xacro:add_transmission joint_name="l_finger_2_joint_1" hardware_interface="${hardware_interface}"/>
-        <xacro:add_transmission joint_name="l_finger_2_joint_2" hardware_interface="${hardware_interface}"/>
-        <xacro:add_transmission joint_name="l_finger_2_joint_3" hardware_interface="${hardware_interface}"/>
-        <xacro:add_transmission joint_name="l_palm_finger_middle_joint" hardware_interface="${hardware_interface}"/>
-        <xacro:add_transmission joint_name="l_finger_middle_joint_1" hardware_interface="${hardware_interface}"/>
-        <xacro:add_transmission joint_name="l_finger_middle_joint_2" hardware_interface="${hardware_interface}"/>
-        <xacro:add_transmission joint_name="l_finger_middle_joint_3" hardware_interface="${hardware_interface}"/>
-        <xacro:add_transmission joint_name="l_finger_1_joint_median_actuating_hinge" hardware_interface="${hardware_interface}"/>
-        <xacro:add_transmission joint_name="l_finger_1_joint_median_actuating_hinge_median_bar" hardware_interface="${hardware_interface}"/>
-        <xacro:add_transmission joint_name="l_finger_1_joint_paradistal_hinge" hardware_interface="${hardware_interface}"/>
-        <xacro:add_transmission joint_name="l_finger_1_joint_paramedian_hinge" hardware_interface="${hardware_interface}"/>
-        <xacro:add_transmission joint_name="l_finger_1_joint_paramedian_hinge_median_bar_underactuated" hardware_interface="${hardware_interface}"/>
-        <xacro:add_transmission joint_name="l_finger_1_joint_paraproximal_actuating_hinge" hardware_interface="${hardware_interface}"/>
-        <xacro:add_transmission joint_name="l_finger_1_joint_paraproximal_bar" hardware_interface="${hardware_interface}"/>
-        <xacro:add_transmission joint_name="l_finger_1_joint_proximal_actuating_bar" hardware_interface="${hardware_interface}"/>
-        <xacro:add_transmission joint_name="l_finger_1_joint_proximal_actuating_hinge" hardware_interface="${hardware_interface}"/>
-        <xacro:add_transmission joint_name="l_finger_2_joint_median_actuating_hinge" hardware_interface="${hardware_interface}"/>
-        <xacro:add_transmission joint_name="l_finger_2_joint_median_actuating_hinge_median_bar" hardware_interface="${hardware_interface}"/>
-        <xacro:add_transmission joint_name="l_finger_2_joint_paradistal_hinge" hardware_interface="${hardware_interface}"/>
-        <xacro:add_transmission joint_name="l_finger_2_joint_paramedian_hinge" hardware_interface="${hardware_interface}"/>
-        <xacro:add_transmission joint_name="l_finger_2_joint_paramedian_hinge_median_bar_underactuated" hardware_interface="${hardware_interface}"/>
-        <xacro:add_transmission joint_name="l_finger_2_joint_paraproximal_actuating_hinge" hardware_interface="${hardware_interface}"/>
-        <xacro:add_transmission joint_name="l_finger_2_joint_paraproximal_bar" hardware_interface="${hardware_interface}"/>
-        <xacro:add_transmission joint_name="l_finger_2_joint_proximal_actuating_bar" hardware_interface="${hardware_interface}"/>
-        <xacro:add_transmission joint_name="l_finger_2_joint_proximal_actuating_hinge" hardware_interface="${hardware_interface}"/>
-        <xacro:add_transmission joint_name="l_finger_middle_joint_median_actuating_hinge" hardware_interface="${hardware_interface}"/>
-        <xacro:add_transmission joint_name="l_finger_middle_joint_median_actuating_hinge_median_bar" hardware_interface="${hardware_interface}"/>
-        <xacro:add_transmission joint_name="l_finger_middle_joint_paradistal_hinge" hardware_interface="${hardware_interface}"/>
-        <xacro:add_transmission joint_name="l_finger_middle_joint_paramedian_hinge" hardware_interface="${hardware_interface}"/>
-        <xacro:add_transmission joint_name="l_finger_middle_joint_paramedian_hinge_median_bar_underactuated" hardware_interface="${hardware_interface}"/>
-        <xacro:add_transmission joint_name="l_finger_middle_joint_paraproximal_actuating_hinge" hardware_interface="${hardware_interface}"/>
-        <xacro:add_transmission joint_name="l_finger_middle_joint_paraproximal_bar" hardware_interface="${hardware_interface}"/>
-        <xacro:add_transmission joint_name="l_finger_middle_joint_proximal_actuating_bar" hardware_interface="${hardware_interface}"/>
-        <xacro:add_transmission joint_name="l_finger_middle_joint_proximal_actuating_hinge" hardware_interface="${hardware_interface}"/>
-        <xacro:add_transmission joint_name="r_finger_1_joint_1" hardware_interface="${hardware_interface}"/>
-        <xacro:add_transmission joint_name="r_finger_1_joint_2" hardware_interface="${hardware_interface}"/>
-        <xacro:add_transmission joint_name="r_finger_1_joint_3" hardware_interface="${hardware_interface}"/>
-        <xacro:add_transmission joint_name="r_finger_1_joint_median_actuating_hinge" hardware_interface="${hardware_interface}"/>
-        <xacro:add_transmission joint_name="r_finger_1_joint_median_actuating_hinge_median_bar" hardware_interface="${hardware_interface}"/>
-        <xacro:add_transmission joint_name="r_finger_1_joint_paradistal_hinge" hardware_interface="${hardware_interface}"/>
-        <xacro:add_transmission joint_name="r_finger_1_joint_paramedian_hinge" hardware_interface="${hardware_interface}"/>
-        <xacro:add_transmission joint_name="r_finger_1_joint_paramedian_hinge_median_bar_underactuated" hardware_interface="${hardware_interface}"/>
-        <xacro:add_transmission joint_name="r_finger_1_joint_paraproximal_actuating_hinge" hardware_interface="${hardware_interface}"/>
-        <xacro:add_transmission joint_name="r_finger_1_joint_paraproximal_bar" hardware_interface="${hardware_interface}"/>
-        <xacro:add_transmission joint_name="r_finger_1_joint_proximal_actuating_bar" hardware_interface="${hardware_interface}"/>
-        <xacro:add_transmission joint_name="r_finger_1_joint_proximal_actuating_hinge" hardware_interface="${hardware_interface}"/>
-        <xacro:add_transmission joint_name="r_finger_2_joint_1" hardware_interface="${hardware_interface}"/>
-        <xacro:add_transmission joint_name="r_finger_2_joint_2" hardware_interface="${hardware_interface}"/>
-        <xacro:add_transmission joint_name="r_finger_2_joint_3" hardware_interface="${hardware_interface}"/>
-        <xacro:add_transmission joint_name="r_finger_2_joint_median_actuating_hinge" hardware_interface="${hardware_interface}"/>
-        <xacro:add_transmission joint_name="r_finger_2_joint_median_actuating_hinge_median_bar" hardware_interface="${hardware_interface}"/>
-        <xacro:add_transmission joint_name="r_finger_2_joint_paradistal_hinge" hardware_interface="${hardware_interface}"/>
-        <xacro:add_transmission joint_name="r_finger_2_joint_paramedian_hinge" hardware_interface="${hardware_interface}"/>
-        <xacro:add_transmission joint_name="r_finger_2_joint_paramedian_hinge_median_bar_underactuated" hardware_interface="${hardware_interface}"/>
-        <xacro:add_transmission joint_name="r_finger_2_joint_paraproximal_actuating_hinge" hardware_interface="${hardware_interface}"/>
-        <xacro:add_transmission joint_name="r_finger_2_joint_paraproximal_bar" hardware_interface="${hardware_interface}"/>
-        <xacro:add_transmission joint_name="r_finger_2_joint_proximal_actuating_bar" hardware_interface="${hardware_interface}"/>
-        <xacro:add_transmission joint_name="r_finger_2_joint_proximal_actuating_hinge" hardware_interface="${hardware_interface}"/>
-        <xacro:add_transmission joint_name="r_finger_middle_joint_1" hardware_interface="${hardware_interface}"/>
-        <xacro:add_transmission joint_name="r_finger_middle_joint_2" hardware_interface="${hardware_interface}"/>
-        <xacro:add_transmission joint_name="r_finger_middle_joint_3" hardware_interface="${hardware_interface}"/>
-        <xacro:add_transmission joint_name="r_finger_middle_joint_median_actuating_hinge" hardware_interface="${hardware_interface}"/>
-        <xacro:add_transmission joint_name="r_finger_middle_joint_median_actuating_hinge_median_bar" hardware_interface="${hardware_interface}"/>
-        <xacro:add_transmission joint_name="r_finger_middle_joint_paradistal_hinge" hardware_interface="${hardware_interface}"/>
-        <xacro:add_transmission joint_name="r_finger_middle_joint_paramedian_hinge" hardware_interface="${hardware_interface}"/>
-        <xacro:add_transmission joint_name="r_finger_middle_joint_paramedian_hinge_median_bar_underactuated" hardware_interface="${hardware_interface}"/>
-        <xacro:add_transmission joint_name="r_finger_middle_joint_paraproximal_actuating_hinge" hardware_interface="${hardware_interface}"/>
-        <xacro:add_transmission joint_name="r_finger_middle_joint_paraproximal_bar" hardware_interface="${hardware_interface}"/>
-        <xacro:add_transmission joint_name="r_finger_middle_joint_proximal_actuating_hinge" hardware_interface="${hardware_interface}"/>
-        <xacro:add_transmission joint_name="r_finger_middle_joint_proximal_actuating_bar" hardware_interface="${hardware_interface}"/>
-        <xacro:add_transmission joint_name="r_palm_finger_1_joint" hardware_interface="${hardware_interface}"/>
-        <xacro:add_transmission joint_name="r_palm_finger_2_joint" hardware_interface="${hardware_interface}"/>
-        <xacro:add_transmission joint_name="r_palm_finger_middle_joint" hardware_interface="${hardware_interface}"/>
+    <xacro:macro name="robotiq_transmissions" params="prefix hardware_interface">
+        <xacro:add_transmission joint_name="${prefix}palm_finger_1_joint"
+                                hardware_interface="${hardware_interface}"/>
+        <xacro:add_transmission joint_name="${prefix}finger_1_joint_1"
+                                hardware_interface="${hardware_interface}"/>
+        <xacro:add_transmission joint_name="${prefix}finger_1_joint_2"
+                                hardware_interface="${hardware_interface}"/>
+        <xacro:add_transmission joint_name="${prefix}finger_1_joint_3"
+                                hardware_interface="${hardware_interface}"/>
+        <xacro:add_transmission joint_name="${prefix}palm_finger_2_joint"
+                                hardware_interface="${hardware_interface}"/>
+        <xacro:add_transmission joint_name="${prefix}finger_2_joint_1"
+                                hardware_interface="${hardware_interface}"/>
+        <xacro:add_transmission joint_name="${prefix}finger_2_joint_2"
+                                hardware_interface="${hardware_interface}"/>
+        <xacro:add_transmission joint_name="${prefix}finger_2_joint_3"
+                                hardware_interface="${hardware_interface}"/>
+        <xacro:add_transmission joint_name="${prefix}palm_finger_middle_joint"
+                                hardware_interface="${hardware_interface}"/>
+        <xacro:add_transmission joint_name="${prefix}finger_middle_joint_1"
+                                hardware_interface="${hardware_interface}"/>
+        <xacro:add_transmission joint_name="${prefix}finger_middle_joint_2"
+                                hardware_interface="${hardware_interface}"/>
+        <xacro:add_transmission joint_name="${prefix}finger_middle_joint_3"
+                                hardware_interface="${hardware_interface}"/>
+        <xacro:add_transmission joint_name="${prefix}finger_1_joint_median_actuating_hinge"
+                                hardware_interface="${hardware_interface}"/>
+        <xacro:add_transmission joint_name="${prefix}finger_1_joint_median_actuating_hinge_median_bar"
+                                hardware_interface="${hardware_interface}"/>
+        <xacro:add_transmission joint_name="${prefix}finger_1_joint_paradistal_hinge"
+                                hardware_interface="${hardware_interface}"/>
+        <xacro:add_transmission joint_name="${prefix}finger_1_joint_paramedian_hinge"
+                                hardware_interface="${hardware_interface}"/>
+        <xacro:add_transmission joint_name="${prefix}finger_1_joint_paramedian_hinge_median_bar_underactuated"
+                                hardware_interface="${hardware_interface}"/>
+        <xacro:add_transmission joint_name="${prefix}finger_1_joint_paraproximal_actuating_hinge"
+                                hardware_interface="${hardware_interface}"/>
+        <xacro:add_transmission joint_name="${prefix}finger_1_joint_paraproximal_bar"
+                                hardware_interface="${hardware_interface}"/>
+        <xacro:add_transmission joint_name="${prefix}finger_1_joint_proximal_actuating_bar"
+                                hardware_interface="${hardware_interface}"/>
+        <xacro:add_transmission joint_name="${prefix}finger_1_joint_proximal_actuating_hinge"
+                                hardware_interface="${hardware_interface}"/>
+        <xacro:add_transmission joint_name="${prefix}finger_2_joint_median_actuating_hinge"
+                                hardware_interface="${hardware_interface}"/>
+        <xacro:add_transmission joint_name="${prefix}finger_2_joint_median_actuating_hinge_median_bar"
+                                hardware_interface="${hardware_interface}"/>
+        <xacro:add_transmission joint_name="${prefix}finger_2_joint_paradistal_hinge"
+                                hardware_interface="${hardware_interface}"/>
+        <xacro:add_transmission joint_name="${prefix}finger_2_joint_paramedian_hinge"
+                                hardware_interface="${hardware_interface}"/>
+        <xacro:add_transmission joint_name="${prefix}finger_2_joint_paramedian_hinge_median_bar_underactuated"
+                                hardware_interface="${hardware_interface}"/>
+        <xacro:add_transmission joint_name="${prefix}finger_2_joint_paraproximal_actuating_hinge"
+                                hardware_interface="${hardware_interface}"/>
+        <xacro:add_transmission joint_name="${prefix}finger_2_joint_paraproximal_bar"
+                                hardware_interface="${hardware_interface}"/>
+        <xacro:add_transmission joint_name="${prefix}finger_2_joint_proximal_actuating_bar"
+                                hardware_interface="${hardware_interface}"/>
+        <xacro:add_transmission joint_name="${prefix}finger_2_joint_proximal_actuating_hinge"
+                                hardware_interface="${hardware_interface}"/>
+        <xacro:add_transmission joint_name="${prefix}finger_middle_joint_median_actuating_hinge"
+                                hardware_interface="${hardware_interface}"/>
+        <xacro:add_transmission joint_name="${prefix}finger_middle_joint_median_actuating_hinge_median_bar"
+                                hardware_interface="${hardware_interface}"/>
+        <xacro:add_transmission joint_name="${prefix}finger_middle_joint_paradistal_hinge"
+                                hardware_interface="${hardware_interface}"/>
+        <xacro:add_transmission joint_name="${prefix}finger_middle_joint_paramedian_hinge"
+                                hardware_interface="${hardware_interface}"/>
+        <xacro:add_transmission joint_name="${prefix}finger_middle_joint_paramedian_hinge_median_bar_underactuated"
+                                hardware_interface="${hardware_interface}"/>
+        <xacro:add_transmission joint_name="${prefix}finger_middle_joint_paraproximal_actuating_hinge"
+                                hardware_interface="${hardware_interface}"/>
+        <xacro:add_transmission joint_name="${prefix}finger_middle_joint_paraproximal_bar"
+                                hardware_interface="${hardware_interface}"/>
+        <xacro:add_transmission joint_name="${prefix}finger_middle_joint_proximal_actuating_bar"
+                                hardware_interface="${hardware_interface}"/>
+        <xacro:add_transmission joint_name="${prefix}finger_middle_joint_proximal_actuating_hinge"
+                                hardware_interface="${hardware_interface}"/>
     </xacro:macro>
 </robot>

File: victor_description/urdf/robotiq_3finger_gripper.xacro (robot description, xacro)
@@ -8,6 +8,6 @@
         <!-- Extensions -->
         <xacro:include filename="$(find victor_description)/urdf/robotiq_3finger_gripper.gazebo.xacro"/>
-        <xacro:include filename="robotiq_3finger_gripper.transmission.xacro"/>
-        <xacro:robotiq_transmissions hardware_interface="${hardware_interface}"/>
+        <xacro:include filename="$(find victor_description)/urdf/robotiq_3finger_gripper.transmission.xacro"/>
+        <xacro:robotiq_transmissions prefix="${prefix}" hardware_interface="${hardware_interface}"/>
     </xacro:macro>
 </robot>
