Commit message: fix mass

File: victor_description/urdf/robotiq_pinch_grasp_tools.xacro (robot description, xacro)
@@ -13,5 +13,5 @@
                 <origin xyz="0 0 0" rpy="0 0 0"/>
                 <!-- It's important that these have non-zero mass, otherwise gazebos URDF to SDF conversion will ignore them -->
-                <mass value="0.00001"/>
+                <mass value="0.001"/>
                 <inertia ixx="0"
                          ixy="0"
@@ -36,5 +36,5 @@
             <inertial>
                 <origin xyz="0 0 0" rpy="0 0 0"/>
-                <mass value="0.00001"/>
+                <mass value="0.001"/>
                 <inertia ixx="0"
                          ixy="0"
