Commit message: Making links and joints squishy in Gazebo.

File: victor_description/urdf/gazebo_utilities.xacro (robot description, xacro)
@@ -1,4 +1,59 @@
 <?xml version="1.0"?>
 <robot xmlns:xacro="http://www.ros.org/wiki/xacro">
+    <xacro:macro name="squishify" params="link_name">
+        <gazebo reference="${link_name}">
+            <collision>
+                <surface>
+                    <bounce>
+                        <restitution_coefficient>0.15</restitution_coefficient>
+                    </bounce>
+                    <contact>
+                        <ode>
+                            <soft_cfm>0.5</soft_cfm>
+                            <soft_erp>0.8</soft_erp>
+                            <kp>100000</kp>
+                            <min_depth>0.0001</min_depth>
+                        </ode>
+                    </contact>
+                </surface>
+            </collision>
+        </gazebo>
+    </xacro:macro>
+    <xacro:macro name="springify" params="joint_name">
+        <gazebo reference="${joint_name}">
+            <axis>
+                <dynamics>
+                    <spring_stiffness>0.1</spring_stiffness>
+                    <spring_reference>0.0</spring_reference>
+                    <damping>0.5</damping>
+                </dynamics>
+            </axis>
+        </gazebo>
+    </xacro:macro>
+    <xacro:macro name="add_simulation_compliance_arm_helper" params="arm index">
+        <xacro:squishify link_name="${arm}_link_${index}"/>
+        <xacro:springify joint_name="${arm}_joint_${index}"/>
+        <xacro:if value="${index-1}">
+            <xacro:add_simulation_compliance_arm_helper arm="${arm}" index="${index-1}"/>
+        </xacro:if>
+        <xacro:unless value="${index-1}">
+            <xacro:squishify link_name="${arm}_link_${index-1}"/>
+        </xacro:unless>
+    </xacro:macro>
+    <xacro:macro name="add_simulation_compliance_finger_helper" params="finger">
+        <xacro:squishify link_name="${finger}_base"/>
+        <xacro:squishify link_name="${finger}_prox"/>
+        <xacro:squishify link_name="${finger}_med"/>
+        <xacro:squishify link_name="${finger}_dist"/>
+        <xacro:springify joint_name="${finger}_joint_2"/>
+        <xacro:springify joint_name="${finger}_joint_3"/>
+        <xacro:springify joint_name="${finger}_joint_4"/>
+    </xacro:macro>
+    <xacro:macro name="add_simulation_compliance" params="side">
+        <xacro:add_simulation_compliance_finger_helper finger="victor_${side}_gripper_fingerA"/>
+        <xacro:add_simulation_compliance_finger_helper finger="victor_${side}_gripper_fingerB"/>
+        <xacro:add_simulation_compliance_finger_helper finger="victor_${side}_gripper_fingerB"/>
+        <xacro:add_simulation_compliance_arm_helper arm="victor_${side}_arm" index="7"/>
+    </xacro:macro>
     <xacro:macro name="add_gazebo_control_plugin" params="robot_namespace">
         <gazebo>
@@ -9,4 +64,15 @@
             </plugin>
         </gazebo>
+        <gazebo> <!-- Unreferenced block is assumed to apply to the robot model -->
+            <!-- Don't forget to update Gazebo path: `export GAZEBO_PLUGIN_PATH=${GAZEBO_PLUGIN_PATH}:~/catkin_ws/devel/lib` -->
+            <plugin name="victor_left_hand_control_plugin" filename="libvictor_gazebo_plugins.so">
+                <side name="left"/>
+            </plugin>
+            <plugin name="victor_right_hand_control_plugin" filename="libvictor_gazebo_plugins.so">
+                <side name="right"/>
+            </plugin>
+        </gazebo>
+        <xacro:add_simulation_compliance side="left"/>
+        <xacro:add_simulation_compliance side="right"/>
     </xacro:macro>
     <xacro:macro name="add_gazebo_fixed_link" params="base_link:=base_link">

File: victor_description/urdf/victor.urdf.xacro (robot description, xacro)
@@ -47,8 +47,8 @@
     <!--Import the Robotiq 3 finger macro -->
     <xacro:include filename="$(find victor_description)/urdf/robotiq_3finger_gripper.xacro"/>
-    <xacro:robotiq_3finger parent="$(arg robot_name)_left_gripper_mounting_bracket" prefix="$(arg robot_name)_left_gripper" hardware_interface="$(arg hardware_interface)">
+    <xacro:robotiq_3finger parent="$(arg robot_name)_left_gripper_mounting_bracket" prefix="$(arg robot_name)_left_gripper" hardware_interface="hardware_interface/EffortJointInterface">
         <origin xyz="0 0 0.02705" rpy="0 0 ${PI/4}"/> <!-- Offset measured with a tape measure; please confirm/fix this value -->
     </xacro:robotiq_3finger>
-    <xacro:robotiq_3finger parent="$(arg robot_name)_right_gripper_mounting_bracket" prefix="$(arg robot_name)_right_gripper" hardware_interface="$(arg hardware_interface)">
+    <xacro:robotiq_3finger parent="$(arg robot_name)_right_gripper_mounting_bracket" prefix="$(arg robot_name)_right_gripper" hardware_interface="hardware_interface/EffortJointInterface">
         <origin xyz="0 0 0.02705" rpy="0 0 ${PI/4}"/> <!-- Offset measured with a tape measure; please confirm/fix this value -->
     </xacro:robotiq_3finger>

Commit message: basic dynamics victor in gazebo
no grippers, very little effort spent tuning PIDs

File: victor_description/urdf/gazebo_utilities.xacro (robot description, xacro)
@@ -59,6 +59,6 @@
         <gazebo>
             <plugin name="gazebo_ros_control" filename="libgazebo_ros_control.so">
-                <!--<robotNamespace>/${robot_namespace}</robotNamespace>-->
-                <robotNamespace>/</robotNamespace>
+                <robotNamespace>/${robot_namespace}</robotNamespace>
+<!--                <robotNamespace>/</robotNamespace>-->
                 <legacyModeNS>false</legacyModeNS>
             </plugin>

File: victor_description/urdf/robotiq_finger.xacro (robot description, xacro)
@@ -1,7 +1,7 @@
 <?xml version="1.0"?>
 <robot xmlns:xacro="http://www.ros.org/wiki/xacro">
-    <xacro:property name="safety_controller_k_pos" value="100"/>
-    <xacro:property name="safety_controller_k_vel" value="100"/>
-    <xacro:property name="joint_damping" value="0.5"/>
+    <xacro:property name="safety_controller_k_pos" value="0"/>
+    <xacro:property name="safety_controller_k_vel" value="0"/>
+    <xacro:property name="joint_damping" value="0.005"/>
     <xacro:property name="max_effort" value="300"/>
     <xacro:property name="max_velocity" value="10"/>
@@ -10,6 +10,6 @@
             <inertial>
                 <origin xyz="0 0 0" rpy="0 0 0"/>
-                <mass value="1"/>
-                <inertia ixx="0.01" ixy="0" ixz="0" iyy="0.01" iyz="0" izz="0.01"/>
+                <mass value="0.1"/>
+                <inertia ixx="0.0001667" ixy="0" ixz="0" iyy="0.0001667" iyz="0" izz="0.0001667"/>
             </inertial>
             <visual>
@@ -45,6 +45,6 @@
             <inertial>
                 <origin xyz="0 0 0" rpy="0 0 0"/>
-                <mass value="1"/>
-                <inertia ixx="0.01" ixy="0" ixz="0" iyy="0.01" iyz="0" izz="0.01"/>
+                <mass value="0.1"/>
+                <inertia ixx="0.0001667" ixy="0" ixz="0" iyy="0.0001667" iyz="0" izz="0.0001667"/>
             </inertial>
             <visual>
@@ -80,6 +80,6 @@
             <inertial>
                 <origin xyz="0 0 0" rpy="0 0 0"/>
-                <mass value="1"/>
-                <inertia ixx="0.01" ixy="0" ixz="0" iyy="0.01" iyz="0" izz="0.01"/>
+                <mass value="0.1"/>
+                <inertia ixx="0.0001667" ixy="0" ixz="0" iyy="0.0001667" iyz="0" izz="0.0001667"/>
             </inertial>
             <visual>
@@ -115,6 +115,6 @@
             <inertial>
                 <origin xyz="0 0 0" rpy="0 0 0"/>
-                <mass value="1"/>
-                <inertia ixx="0.01" ixy="0" ixz="0" iyy="0.01" iyz="0" izz="0.01"/>
+                <mass value="0.1"/>
+                <inertia ixx="0.0001667" ixy="0" ixz="0" iyy="0.0001667" iyz="0" izz="0.0001667"/>
             </inertial>
             <visual>

File: victor_description/urdf/victor.urdf.xacro (robot description, xacro)
@@ -53,42 +53,4 @@
         <origin xyz="0 0 0.02705" rpy="0 0 ${PI/4}"/> <!-- Offset measured with a tape measure; please confirm/fix this value -->
     </xacro:robotiq_3finger>
-    <link name="$(arg robot_name)_left_tool_placeholder">
-        <visual>
-            <origin xyz="0 0 0" rpy="0 0 0"/>
-            <geometry>
-                <cylinder length="${6 * 0.0254}" radius="0.03"/>
-            </geometry>
-        </visual>
-        <collision>
-            <origin xyz="0 0 0" rpy="0 0 0"/>
-            <geometry>
-                <cylinder length="${6 * 0.0254}" radius="0.03"/>
-            </geometry>
-        </collision>
-    </link>
-    <joint name="$(arg robot_name)_left_tool_joint" type="fixed">
-        <parent link="$(arg robot_name)_left_gripper_palm_surface"/>
-        <child link="$(arg robot_name)_left_tool_placeholder"/>
-        <origin xyz="0 0 ${3 * 0.0254}"/>
-    </joint>
-    <link name="$(arg robot_name)_right_tool_placeholder">
-        <visual>
-            <origin xyz="0 0 0" rpy="0 0 0"/>
-            <geometry>
-                <cylinder length="${6 * 0.0254}" radius="0.03"/>
-            </geometry>
-        </visual>
-        <collision>
-            <origin xyz="0 0 0" rpy="0 0 0"/>
-            <geometry>
-                <cylinder length="${6 * 0.0254}" radius="0.03"/>
-            </geometry>
-        </collision>
-    </link>
-    <joint name="$(arg robot_name)_right_tool_joint" type="fixed">
-        <parent link="$(arg robot_name)_right_gripper_palm_surface"/>
-        <child link="$(arg robot_name)_right_tool_placeholder"/>
-        <origin xyz="0 0 ${3 * 0.0254}"/>
-    </joint>
     <!-- Add Gazebo properties for whole robot -->
     <xacro:include filename="$(find victor_description)/urdf/gazebo_utilities.xacro"/>
@@ -96,4 +58,4 @@
     <xacro:add_gazebo_control_plugin robot_namespace="$(arg robot_name)"/>
     <!-- Rigidly attach Victor to the Gazebo world -->
-    <!-- <xacro:add_gazebo_fixed_link base_link="$(arg robot_name)_root"/> -->
+    <xacro:add_gazebo_fixed_link base_link="$(arg robot_name)_root"/>
 </robot>

Commit message: add back the fake tool stuff

File: victor_description/urdf/gazebo_utilities.xacro (robot description, xacro)
@@ -59,6 +59,6 @@
         <gazebo>
             <plugin name="gazebo_ros_control" filename="libgazebo_ros_control.so">
-                <robotNamespace>/${robot_namespace}</robotNamespace>
-<!--                <robotNamespace>/</robotNamespace>-->
+                <!--<robotNamespace>/${robot_namespace}</robotNamespace>-->
+                <robotNamespace>/</robotNamespace>
                 <legacyModeNS>false</legacyModeNS>
             </plugin>

File: victor_description/urdf/victor.urdf.xacro (robot description, xacro)
@@ -53,4 +53,42 @@
         <origin xyz="0 0 0.02705" rpy="0 0 ${PI/4}"/> <!-- Offset measured with a tape measure; please confirm/fix this value -->
     </xacro:robotiq_3finger>
+    <link name="$(arg robot_name)_left_tool_placeholder">
+        <visual>
+            <origin xyz="0 0 0" rpy="0 0 0"/>
+            <geometry>
+                <cylinder length="${6 * 0.0254}" radius="0.03"/>
+            </geometry>
+        </visual>
+        <collision>
+            <origin xyz="0 0 0" rpy="0 0 0"/>
+            <geometry>
+                <cylinder length="${6 * 0.0254}" radius="0.03"/>
+            </geometry>
+        </collision>
+    </link>
+    <joint name="$(arg robot_name)_left_tool_joint" type="fixed">
+        <parent link="$(arg robot_name)_left_gripper_palm_surface"/>
+        <child link="$(arg robot_name)_left_tool_placeholder"/>
+        <origin xyz="0 0 ${3 * 0.0254}"/>
+    </joint>
+    <link name="$(arg robot_name)_right_tool_placeholder">
+        <visual>
+            <origin xyz="0 0 0" rpy="0 0 0"/>
+            <geometry>
+                <cylinder length="${6 * 0.0254}" radius="0.03"/>
+            </geometry>
+        </visual>
+        <collision>
+            <origin xyz="0 0 0" rpy="0 0 0"/>
+            <geometry>
+                <cylinder length="${6 * 0.0254}" radius="0.03"/>
+            </geometry>
+        </collision>
+    </link>
+    <joint name="$(arg robot_name)_right_tool_joint" type="fixed">
+        <parent link="$(arg robot_name)_right_gripper_palm_surface"/>
+        <child link="$(arg robot_name)_right_tool_placeholder"/>
+        <origin xyz="0 0 ${3 * 0.0254}"/>
+    </joint>
     <!-- Add Gazebo properties for whole robot -->
     <xacro:include filename="$(find victor_description)/urdf/gazebo_utilities.xacro"/>
@@ -58,4 +96,4 @@
     <xacro:add_gazebo_control_plugin robot_namespace="$(arg robot_name)"/>
     <!-- Rigidly attach Victor to the Gazebo world -->
-    <xacro:add_gazebo_fixed_link base_link="$(arg robot_name)_root"/>
+    <!-- <xacro:add_gazebo_fixed_link base_link="$(arg robot_name)_root"/> -->
 </robot>

Commit message: change srdf to make more sense to me
rename tool frames to be robot generic

File: victor_description/urdf/gazebo_utilities.xacro (robot description, xacro)
@@ -1,4 +1,46 @@
 <?xml version="1.0"?>
 <robot xmlns:xacro="http://www.ros.org/wiki/xacro">
+    <gazebo reference="victor_right_arm_link_1">
+        <self_collide>1</self_collide>
+    </gazebo>
+    <gazebo reference="victor_right_arm_link_2">
+        <self_collide>1</self_collide>
+    </gazebo>
+    <gazebo reference="victor_right_arm_link_3">
+        <self_collide>1</self_collide>
+    </gazebo>
+    <gazebo reference="victor_right_arm_link_4">
+        <self_collide>1</self_collide>
+    </gazebo>
+    <gazebo reference="victor_right_arm_link_5">
+        <self_collide>1</self_collide>
+    </gazebo>
+    <gazebo reference="victor_right_arm_link_6">
+        <self_collide>1</self_collide>
+    </gazebo>
+    <gazebo reference="victor_right_arm_link_7">
+        <self_collide>0</self_collide>
+    </gazebo>
+    <gazebo reference="victor_left_arm_link_1">
+        <self_collide>1</self_collide>
+    </gazebo>
+    <gazebo reference="victor_left_arm_link_2">
+        <self_collide>1</self_collide>
+    </gazebo>
+    <gazebo reference="victor_left_arm_link_3">
+        <self_collide>1</self_collide>
+    </gazebo>
+    <gazebo reference="victor_left_arm_link_4">
+        <self_collide>1</self_collide>
+    </gazebo>
+    <gazebo reference="victor_left_arm_link_5">
+        <self_collide>1</self_collide>
+    </gazebo>
+    <gazebo reference="victor_left_arm_link_6">
+        <self_collide>1</self_collide>
+    </gazebo>
+    <gazebo reference="victor_left_arm_link_7">
+        <self_collide>0</self_collide>
+    </gazebo>
     <xacro:macro name="squishify" params="link_name">
         <gazebo reference="${link_name}">
@@ -60,5 +102,5 @@
             <plugin name="gazebo_ros_control" filename="libgazebo_ros_control.so">
                 <robotNamespace>/${robot_namespace}</robotNamespace>
-<!--                <robotNamespace>/</robotNamespace>-->
+                <!--                <robotNamespace>/</robotNamespace>-->
                 <legacyModeNS>false</legacyModeNS>
             </plugin>
@@ -77,9 +119,9 @@
     </xacro:macro>
     <xacro:macro name="add_gazebo_fixed_link" params="base_link:=base_link">
-        <link name="world" />
+        <link name="world"/>
         <joint name="world_joint" type="fixed">
-            <parent link="world" />
-            <child link = "${base_link}" />
-            <origin xyz="0.0 0.0 0.0" rpy="0.0 0.0 0.0" />
+            <parent link="world"/>
+            <child link="${base_link}"/>
+            <origin xyz="0.0 0.0 0.0" rpy="0.0 0.0 0.0"/>
         </joint>
     </xacro:macro>

Commit message: reorganize xacro macros so I can use some of them in HDT

File: victor_description/urdf/gazebo_utilities.xacro (robot description, xacro)
@@ -1,64 +1,4 @@
 <?xml version="1.0"?>
 <robot xmlns:xacro="http://www.ros.org/wiki/xacro">
-    <gazebo reference="victor_right_arm_link_1">
-        <self_collide>1</self_collide>
-    </gazebo>
-    <gazebo reference="victor_right_arm_link_2">
-        <self_collide>1</self_collide>
-    </gazebo>
-    <gazebo reference="victor_right_arm_link_3">
-        <self_collide>1</self_collide>
-    </gazebo>
-    <gazebo reference="victor_right_arm_link_4">
-        <self_collide>1</self_collide>
-    </gazebo>
-    <gazebo reference="victor_right_arm_link_5">
-        <self_collide>1</self_collide>
-    </gazebo>
-    <gazebo reference="victor_right_arm_link_6">
-        <self_collide>1</self_collide>
-    </gazebo>
-    <gazebo reference="victor_right_arm_link_7">
-        <self_collide>0</self_collide>
-    </gazebo>
-    <gazebo reference="victor_right_gripper_fingerA_dist">
-        <self_collide>1</self_collide>
-    </gazebo>
-    <gazebo reference="victor_right_gripper_fingerB_dist">
-        <self_collide>1</self_collide>
-    </gazebo>
-    <gazebo reference="victor_right_gripper_fingerC_dist">
-        <self_collide>1</self_collide>
-    </gazebo>
-    <gazebo reference="victor_left_arm_link_1">
-        <self_collide>1</self_collide>
-    </gazebo>
-    <gazebo reference="victor_left_arm_link_2">
-        <self_collide>1</self_collide>
-    </gazebo>
-    <gazebo reference="victor_left_arm_link_3">
-        <self_collide>1</self_collide>
-    </gazebo>
-    <gazebo reference="victor_left_arm_link_4">
-        <self_collide>1</self_collide>
-    </gazebo>
-    <gazebo reference="victor_left_arm_link_5">
-        <self_collide>1</self_collide>
-    </gazebo>
-    <gazebo reference="victor_left_arm_link_6">
-        <self_collide>1</self_collide>
-    </gazebo>
-    <gazebo reference="victor_left_arm_link_7">
-        <self_collide>0</self_collide>
-    </gazebo>
-    <gazebo reference="victor_left_gripper_fingerA_dist">
-        <self_collide>1</self_collide>
-    </gazebo>
-    <gazebo reference="victor_left_gripper_fingerB_dist">
-        <self_collide>1</self_collide>
-    </gazebo>
-    <gazebo reference="victor_left_gripper_fingerC_dist">
-        <self_collide>1</self_collide>
-    </gazebo>
     <xacro:macro name="squishify" params="link_name">
         <gazebo reference="${link_name}">
@@ -110,20 +50,20 @@
         <xacro:springify joint_name="${finger}_joint_4"/>
     </xacro:macro>
-    <xacro:macro name="add_simulation_compliance" params="side">
-        <xacro:add_simulation_compliance_finger_helper finger="victor_${side}_gripper_fingerA"/>
-        <xacro:add_simulation_compliance_finger_helper finger="victor_${side}_gripper_fingerB"/>
-        <xacro:add_simulation_compliance_finger_helper finger="victor_${side}_gripper_fingerB"/>
-        <xacro:add_simulation_compliance_arm_helper arm="victor_${side}_arm" index="7"/>
-    </xacro:macro>
     <xacro:macro name="add_gazebo_control_plugin" params="robot_namespace">
         <gazebo>
             <plugin name="gazebo_ros_control" filename="libgazebo_ros_control.so">
-                <robotNamespace>/${robot_namespace}</robotNamespace>
-                <!--                <robotNamespace>/</robotNamespace>-->
+                <robotNamespace>${robot_namespace}</robotNamespace>
                 <legacyModeNS>false</legacyModeNS>
             </plugin>
         </gazebo>
-        <xacro:add_simulation_compliance side="left"/>
-        <xacro:add_simulation_compliance side="right"/>
+    </xacro:macro>
+    <xacro:macro name="add_moveit_planning_scene_plugin" params="robot_namespace root_frame_id">
+        <gazebo>
+            <plugin name="gazebo_ros_moveit_planning_scene" filename="libgazebo_ros_moveit_planning_scene.so">
+                <robotName>${robot_namespace}</robotName>
+                <!--  This must be the same as the root frame of the robot you're using -->
+                <frameId>${root_frame_id}</frameId>
+            </plugin>
+        </gazebo>
     </xacro:macro>
     <xacro:macro name="add_gazebo_fixed_link" params="base_link:=base_link">

File: victor_description/urdf/victor.urdf.xacro (robot description, xacro)
@@ -47,8 +47,10 @@
     <!--Import the Robotiq 3 finger macro -->
     <xacro:include filename="$(find victor_description)/urdf/robotiq_3finger_gripper.xacro"/>
-    <xacro:robotiq_3finger parent="$(arg robot_name)_left_gripper_mounting_bracket" prefix="$(arg robot_name)_left_gripper" hardware_interface="$(arg hardware_interface)">
+    <xacro:robotiq_3finger parent="$(arg robot_name)_left_gripper_mounting_bracket" prefix="$(arg robot_name)_left_gripper"
+                           hardware_interface="$(arg hardware_interface)">
         <origin xyz="0 0 0.02705" rpy="0 0 ${PI/4}"/> <!-- Offset measured with a tape measure; please confirm/fix this value -->
     </xacro:robotiq_3finger>
-    <xacro:robotiq_3finger parent="$(arg robot_name)_right_gripper_mounting_bracket" prefix="$(arg robot_name)_right_gripper" hardware_interface="$(arg hardware_interface)">
+    <xacro:robotiq_3finger parent="$(arg robot_name)_right_gripper_mounting_bracket" prefix="$(arg robot_name)_right_gripper"
+                           hardware_interface="$(arg hardware_interface)">
         <origin xyz="0 0 0.02705" rpy="0 0 ${PI/4}"/> <!-- Offset measured with a tape measure; please confirm/fix this value -->
     </xacro:robotiq_3finger>
@@ -57,7 +59,10 @@
     <xacro:robotiq_pinch_grasp_tools robot_name="$(arg robot_name)"/>
     <!-- Add Gazebo properties for whole robot -->
+    <xacro:include filename="$(find victor_description)/urdf/victor.gazebo.xacro"/>
     <xacro:include filename="$(find victor_description)/urdf/gazebo_utilities.xacro"/>
     <!-- Load Gazebo lib and set the robot namespace -->
     <xacro:add_gazebo_control_plugin robot_namespace="$(arg robot_name)"/>
+    <xacro:add_simulation_compliance side="left"/>
+    <xacro:add_simulation_compliance side="right"/>
     <!-- Rigidly attach Victor to the Gazebo world -->
     <xacro:add_gazebo_fixed_link base_link="$(arg robot_name)_root"/>
