Commit message: change namespacing
trying to understand how to make the jacobian motion smooth
the position controllers seem really smooth when doing joint space plans
I think we need to include velocity/postion in the waypoints somehow

File: victor_description/urdf/gazebo_utilities.xacro (robot description, xacro)
@@ -66,5 +66,5 @@
                 <frameId>${root_frame_id}</frameId>
                 <excludedModels>collision_sphere</excludedModels>
-                <scalePrimitivesFactor>1.2</scalePrimitivesFactor>
+                <scalePrimitivesFactor>1.0</scalePrimitivesFactor>
             </plugin>
         </gazebo>
@@ -78,3 +78,13 @@
         </joint>
     </xacro:macro>
+    <xacro:macro name="add_joint_cfm_damping" params="joint_name cfm_damping">
+        <gazebo reference="${joint_name}">
+            <physics>
+                <ode>
+                    <cfm>0.01</cfm>
+                    <implicit_spring_damper>1</implicit_spring_damper>
+                </ode>
+            </physics>
+        </gazebo>
+    </xacro:macro>
 </robot>

File: victor_description/urdf/robotiq_3finger_gripper.xacro (robot description, xacro)
@@ -4,4 +4,5 @@
     <xacro:include filename="$(find victor_description)/urdf/robotiq_3finger_gripper.transmission.xacro"/>
     <xacro:macro name="robotiq_3finger" params="parent prefix hardware_interface *origin">
+        <xacro:property name="joint_damping" value="0.05"/>
         <joint name="${prefix}_palm_joint" type="fixed">
             <xacro:insert_block name="origin"/>
@@ -52,5 +53,5 @@
             <child link="${prefix}_fingerA_base"/>
         </joint>
-        <xacro:robotiq_finger prefix="${prefix}_fingerA"/>
+        <xacro:robotiq_finger prefix="${prefix}_fingerA" joint_damping="${joint_damping}"/>
         <!-- Finger B -->
         <joint name="${prefix}_fingerB_knuckle" type="revolute">
@@ -63,5 +64,5 @@
             <dynamics damping="${joint_damping}"/>
         </joint>
-        <xacro:robotiq_finger prefix="${prefix}_fingerB"/>
+        <xacro:robotiq_finger prefix="${prefix}_fingerB" joint_damping="${joint_damping}"/>
         <!-- Finger C -->
         <joint name="${prefix}_fingerC_knuckle" type="revolute">
@@ -74,5 +75,5 @@
             <dynamics damping="${joint_damping}"/>
         </joint>
-        <xacro:robotiq_finger prefix="${prefix}_fingerC"/>
+        <xacro:robotiq_finger prefix="${prefix}_fingerC" joint_damping="${joint_damping}"/>
         <xacro:robotiq_3finger_gripper_transmission hardware_interface="${hardware_interface}"
                                                     robot_name="${prefix}"/>

File: victor_description/urdf/robotiq_finger.xacro (robot description, xacro)
@@ -1,8 +1,7 @@
 <?xml version="1.0"?>
 <robot xmlns:xacro="http://www.ros.org/wiki/xacro">
-    <xacro:property name="joint_damping" value="0.005"/>
     <xacro:property name="max_effort" value="300"/>
     <xacro:property name="max_velocity" value="10"/>
-    <xacro:macro name="robotiq_finger" params="prefix">
+    <xacro:macro name="robotiq_finger" params="prefix joint_damping">
         <link name="${prefix}_base">
             <inertial>

File: victor_description/urdf/victor.urdf.xacro (robot description, xacro)
@@ -63,4 +63,5 @@
     <!-- Load Gazebo lib and set the robot namespace -->
     <xacro:add_gazebo_control_plugin robot_namespace="$(arg robot_name)"/>
+    <xacro:add_moveit_planning_scene_plugin robot_namespace="$(arg robot_name)" root_frame_id="victor_root"/>
     <xacro:add_simulation_compliance side="left"/>
     <xacro:add_simulation_compliance side="right"/>
