Commit message: new grippers in the right spot
the srdf files is a disaster

File: victor_description/urdf/gazebo_utilities.xacro (robot description, xacro)
@@ -88,3 +88,14 @@
         </gazebo>
     </xacro:macro>
+    <xacro:macro name="add_transmission" params="joint_name hardware_interface">
+        <transmission name="${joint_name}_tran">
+            <type>transmission_interface/SimpleTransmission</type>
+            <joint name="${joint_name}">
+                <hardwareInterface>${hardware_interface}</hardwareInterface>
+            </joint>
+            <actuator name="${joint_name}_motor">
+                <mechanicalReduction>1</mechanicalReduction>
+            </actuator>
+        </transmission>
+    </xacro:macro>
 </robot>

File: victor_description/urdf/robotiq_3finger_gripper.transmission.xacro (robot description, xacro)
@@ -1,104 +1,84 @@
 <?xml version="1.0"?>
 <robot xmlns:xacro="http://www.ros.org/wiki/xacro">
-  <xacro:macro name="robotiq_3finger_gripper_transmission" params="hardware_interface robot_name">
-    <transmission name="${robot_name}_tran_A2">
-      <type>transmission_interface/SimpleTransmission</type>
-      <joint name="${robot_name}_fingerA_joint_2">
-        <hardwareInterface>${hardware_interface}</hardwareInterface>
-      </joint>
-      <actuator name="${robot_name}_motor_A2">
-        <mechanicalReduction>1</mechanicalReduction>
-      </actuator>
-    </transmission>
-    <transmission name="${robot_name}_tran_A3">
-      <type>transmission_interface/SimpleTransmission</type>
-      <joint name="${robot_name}_fingerA_joint_3">
-        <hardwareInterface>${hardware_interface}</hardwareInterface>
-      </joint>
-      <actuator name="${robot_name}_motor_A3">
-        <mechanicalReduction>1</mechanicalReduction>
-      </actuator>
-    </transmission>
-    <transmission name="${robot_name}_tran_A4">
-      <type>transmission_interface/SimpleTransmission</type>
-      <joint name="${robot_name}_fingerA_joint_4">
-        <hardwareInterface>${hardware_interface}</hardwareInterface>
-      </joint>
-      <actuator name="${robot_name}_motor_A4">
-        <mechanicalReduction>1</mechanicalReduction>
-      </actuator>
-    </transmission>
-    <transmission name="${robot_name}_tran_B2">
-      <type>transmission_interface/SimpleTransmission</type>
-      <joint name="${robot_name}_fingerB_joint_2">
-        <hardwareInterface>${hardware_interface}</hardwareInterface>
-      </joint>
-      <actuator name="${robot_name}_motor_B2">
-        <mechanicalReduction>1</mechanicalReduction>
-      </actuator>
-    </transmission>
-    <transmission name="${robot_name}_tran_B3">
-      <type>transmission_interface/SimpleTransmission</type>
-      <joint name="${robot_name}_fingerB_joint_3">
-        <hardwareInterface>${hardware_interface}</hardwareInterface>
-      </joint>
-      <actuator name="${robot_name}_motor_B3">
-        <mechanicalReduction>1</mechanicalReduction>
-      </actuator>
-    </transmission>
-    <transmission name="${robot_name}_tran_B4">
-      <type>transmission_interface/SimpleTransmission</type>
-      <joint name="${robot_name}_fingerB_joint_4">
-        <hardwareInterface>${hardware_interface}</hardwareInterface>
-      </joint>
-      <actuator name="${robot_name}_motor_B4">
-        <mechanicalReduction>1</mechanicalReduction>
-      </actuator>
-    </transmission>
-    <transmission name="${robot_name}_tran_C2">
-      <type>transmission_interface/SimpleTransmission</type>
-      <joint name="${robot_name}_fingerC_joint_2">
-        <hardwareInterface>${hardware_interface}</hardwareInterface>
-      </joint>
-      <actuator name="${robot_name}_motor_C2">
-        <mechanicalReduction>1</mechanicalReduction>
-      </actuator>
-    </transmission>
-    <transmission name="${robot_name}_tran_C3">
-      <type>transmission_interface/SimpleTransmission</type>
-      <joint name="${robot_name}_fingerC_joint_3">
-        <hardwareInterface>${hardware_interface}</hardwareInterface>
-      </joint>
-      <actuator name="${robot_name}_motor_C3">
-        <mechanicalReduction>1</mechanicalReduction>
-      </actuator>
-    </transmission>
-    <transmission name="${robot_name}_tran_C4">
-      <type>transmission_interface/SimpleTransmission</type>
-      <joint name="${robot_name}_fingerC_joint_4">
-        <hardwareInterface>${hardware_interface}</hardwareInterface>
-      </joint>
-      <actuator name="${robot_name}_motor_C4">
-        <mechanicalReduction>1</mechanicalReduction>
-      </actuator>
-    </transmission>
-    <transmission name="${robot_name}_tran_Bknuckle">
-      <type>transmission_interface/SimpleTransmission</type>
-      <joint name="${robot_name}_fingerB_knuckle">
-        <hardwareInterface>${hardware_interface}</hardwareInterface>
-      </joint>
-      <actuator name="${robot_name}_motor_Bknuckle">
-        <mechanicalReduction>1</mechanicalReduction>
-      </actuator>
-    </transmission>
-    <transmission name="${robot_name}_tran_Cknuckle">
-      <type>transmission_interface/SimpleTransmission</type>
-      <joint name="${robot_name}_fingerC_knuckle">
-        <hardwareInterface>${hardware_interface}</hardwareInterface>
-      </joint>
-      <actuator name="${robot_name}_motor_Cknuckle">
-        <mechanicalReduction>1</mechanicalReduction>
-      </actuator>
-    </transmission>
-  </xacro:macro>
+    <xacro:include filename="$(find victor_description)/urdf/gazebo_utilities.xacro"/>
+    <xacro:macro name="robotiq_transmissions" params="hardware_interface">
+        <xacro:add_transmission joint_name="l_palm_finger_1_joint" hardware_interface="${hardware_interface}"/>
+        <xacro:add_transmission joint_name="l_finger_1_joint_1" hardware_interface="${hardware_interface}"/>
+        <xacro:add_transmission joint_name="l_finger_1_joint_2" hardware_interface="${hardware_interface}"/>
+        <xacro:add_transmission joint_name="l_finger_1_joint_3" hardware_interface="${hardware_interface}"/>
+        <xacro:add_transmission joint_name="l_palm_finger_2_joint" hardware_interface="${hardware_interface}"/>
+        <xacro:add_transmission joint_name="l_finger_2_joint_1" hardware_interface="${hardware_interface}"/>
+        <xacro:add_transmission joint_name="l_finger_2_joint_2" hardware_interface="${hardware_interface}"/>
+        <xacro:add_transmission joint_name="l_finger_2_joint_3" hardware_interface="${hardware_interface}"/>
+        <xacro:add_transmission joint_name="l_palm_finger_middle_joint" hardware_interface="${hardware_interface}"/>
+        <xacro:add_transmission joint_name="l_finger_middle_joint_1" hardware_interface="${hardware_interface}"/>
+        <xacro:add_transmission joint_name="l_finger_middle_joint_2" hardware_interface="${hardware_interface}"/>
+        <xacro:add_transmission joint_name="l_finger_middle_joint_3" hardware_interface="${hardware_interface}"/>
+        <xacro:add_transmission joint_name="l_finger_1_joint_median_actuating_hinge" hardware_interface="${hardware_interface}"/>
+        <xacro:add_transmission joint_name="l_finger_1_joint_median_actuating_hinge_median_bar" hardware_interface="${hardware_interface}"/>
+        <xacro:add_transmission joint_name="l_finger_1_joint_paradistal_hinge" hardware_interface="${hardware_interface}"/>
+        <xacro:add_transmission joint_name="l_finger_1_joint_paramedian_hinge" hardware_interface="${hardware_interface}"/>
+        <xacro:add_transmission joint_name="l_finger_1_joint_paramedian_hinge_median_bar_underactuated" hardware_interface="${hardware_interface}"/>
+        <xacro:add_transmission joint_name="l_finger_1_joint_paraproximal_actuating_hinge" hardware_interface="${hardware_interface}"/>
+        <xacro:add_transmission joint_name="l_finger_1_joint_paraproximal_bar" hardware_interface="${hardware_interface}"/>
+        <xacro:add_transmission joint_name="l_finger_1_joint_proximal_actuating_bar" hardware_interface="${hardware_interface}"/>
+        <xacro:add_transmission joint_name="l_finger_1_joint_proximal_actuating_hinge" hardware_interface="${hardware_interface}"/>
+        <xacro:add_transmission joint_name="l_finger_2_joint_median_actuating_hinge" hardware_interface="${hardware_interface}"/>
+        <xacro:add_transmission joint_name="l_finger_2_joint_median_actuating_hinge_median_bar" hardware_interface="${hardware_interface}"/>
+        <xacro:add_transmission joint_name="l_finger_2_joint_paradistal_hinge" hardware_interface="${hardware_interface}"/>
+        <xacro:add_transmission joint_name="l_finger_2_joint_paramedian_hinge" hardware_interface="${hardware_interface}"/>
+        <xacro:add_transmission joint_name="l_finger_2_joint_paramedian_hinge_median_bar_underactuated" hardware_interface="${hardware_interface}"/>
+        <xacro:add_transmission joint_name="l_finger_2_joint_paraproximal_actuating_hinge" hardware_interface="${hardware_interface}"/>
+        <xacro:add_transmission joint_name="l_finger_2_joint_paraproximal_bar" hardware_interface="${hardware_interface}"/>
+        <xacro:add_transmission joint_name="l_finger_2_joint_proximal_actuating_bar" hardware_interface="${hardware_interface}"/>
+        <xacro:add_transmission joint_name="l_finger_2_joint_proximal_actuating_hinge" hardware_interface="${hardware_interface}"/>
+        <xacro:add_transmission joint_name="l_finger_middle_joint_median_actuating_hinge" hardware_interface="${hardware_interface}"/>
+        <xacro:add_transmission joint_name="l_finger_middle_joint_median_actuating_hinge_median_bar" hardware_interface="${hardware_interface}"/>
+        <xacro:add_transmission joint_name="l_finger_middle_joint_paradistal_hinge" hardware_interface="${hardware_interface}"/>
+        <xacro:add_transmission joint_name="l_finger_middle_joint_paramedian_hinge" hardware_interface="${hardware_interface}"/>
+        <xacro:add_transmission joint_name="l_finger_middle_joint_paramedian_hinge_median_bar_underactuated" hardware_interface="${hardware_interface}"/>
+        <xacro:add_transmission joint_name="l_finger_middle_joint_paraproximal_actuating_hinge" hardware_interface="${hardware_interface}"/>
+        <xacro:add_transmission joint_name="l_finger_middle_joint_paraproximal_bar" hardware_interface="${hardware_interface}"/>
+        <xacro:add_transmission joint_name="l_finger_middle_joint_proximal_actuating_bar" hardware_interface="${hardware_interface}"/>
+        <xacro:add_transmission joint_name="l_finger_middle_joint_proximal_actuating_hinge" hardware_interface="${hardware_interface}"/>
+        <xacro:add_transmission joint_name="r_finger_1_joint_1" hardware_interface="${hardware_interface}"/>
+        <xacro:add_transmission joint_name="r_finger_1_joint_2" hardware_interface="${hardware_interface}"/>
+        <xacro:add_transmission joint_name="r_finger_1_joint_3" hardware_interface="${hardware_interface}"/>
+        <xacro:add_transmission joint_name="r_finger_1_joint_median_actuating_hinge" hardware_interface="${hardware_interface}"/>
+        <xacro:add_transmission joint_name="r_finger_1_joint_median_actuating_hinge_median_bar" hardware_interface="${hardware_interface}"/>
+        <xacro:add_transmission joint_name="r_finger_1_joint_paradistal_hinge" hardware_interface="${hardware_interface}"/>
+        <xacro:add_transmission joint_name="r_finger_1_joint_paramedian_hinge" hardware_interface="${hardware_interface}"/>
+        <xacro:add_transmission joint_name="r_finger_1_joint_paramedian_hinge_median_bar_underactuated" hardware_interface="${hardware_interface}"/>
+        <xacro:add_transmission joint_name="r_finger_1_joint_paraproximal_actuating_hinge" hardware_interface="${hardware_interface}"/>
+        <xacro:add_transmission joint_name="r_finger_1_joint_paraproximal_bar" hardware_interface="${hardware_interface}"/>
+        <xacro:add_transmission joint_name="r_finger_1_joint_proximal_actuating_bar" hardware_interface="${hardware_interface}"/>
+        <xacro:add_transmission joint_name="r_finger_1_joint_proximal_actuating_hinge" hardware_interface="${hardware_interface}"/>
+        <xacro:add_transmission joint_name="r_finger_2_joint_1" hardware_interface="${hardware_interface}"/>
+        <xacro:add_transmission joint_name="r_finger_2_joint_2" hardware_interface="${hardware_interface}"/>
+        <xacro:add_transmission joint_name="r_finger_2_joint_3" hardware_interface="${hardware_interface}"/>
+        <xacro:add_transmission joint_name="r_finger_2_joint_median_actuating_hinge" hardware_interface="${hardware_interface}"/>
+        <xacro:add_transmission joint_name="r_finger_2_joint_median_actuating_hinge_median_bar" hardware_interface="${hardware_interface}"/>
+        <xacro:add_transmission joint_name="r_finger_2_joint_paradistal_hinge" hardware_interface="${hardware_interface}"/>
+        <xacro:add_transmission joint_name="r_finger_2_joint_paramedian_hinge" hardware_interface="${hardware_interface}"/>
+        <xacro:add_transmission joint_name="r_finger_2_joint_paramedian_hinge_median_bar_underactuated" hardware_interface="${hardware_interface}"/>
+        <xacro:add_transmission joint_name="r_finger_2_joint_paraproximal_actuating_hinge" hardware_interface="${hardware_interface}"/>
+        <xacro:add_transmission joint_name="r_finger_2_joint_paraproximal_bar" hardware_interface="${hardware_interface}"/>
+        <xacro:add_transmission joint_name="r_finger_2_joint_proximal_actuating_bar" hardware_interface="${hardware_interface}"/>
+        <xacro:add_transmission joint_name="r_finger_2_joint_proximal_actuating_hinge" hardware_interface="${hardware_interface}"/>
+        <xacro:add_transmission joint_name="r_finger_middle_joint_1" hardware_interface="${hardware_interface}"/>
+        <xacro:add_transmission joint_name="r_finger_middle_joint_2" hardware_interface="${hardware_interface}"/>
+        <xacro:add_transmission joint_name="r_finger_middle_joint_3" hardware_interface="${hardware_interface}"/>
+        <xacro:add_transmission joint_name="r_finger_middle_joint_median_actuating_hinge" hardware_interface="${hardware_interface}"/>
+        <xacro:add_transmission joint_name="r_finger_middle_joint_median_actuating_hinge_median_bar" hardware_interface="${hardware_interface}"/>
+        <xacro:add_transmission joint_name="r_finger_middle_joint_paradistal_hinge" hardware_interface="${hardware_interface}"/>
+        <xacro:add_transmission joint_name="r_finger_middle_joint_paramedian_hinge" hardware_interface="${hardware_interface}"/>
+        <xacro:add_transmission joint_name="r_finger_middle_joint_paramedian_hinge_median_bar_underactuated" hardware_interface="${hardware_interface}"/>
+        <xacro:add_transmission joint_name="r_finger_middle_joint_paraproximal_actuating_hinge" hardware_interface="${hardware_interface}"/>
+        <xacro:add_transmission joint_name="r_finger_middle_joint_paraproximal_bar" hardware_interface="${hardware_interface}"/>
+        <xacro:add_transmission joint_name="r_finger_middle_joint_proximal_actuating_hinge" hardware_interface="${hardware_interface}"/>
+        <xacro:add_transmission joint_name="r_finger_middle_joint_proximal_actuating_bar" hardware_interface="${hardware_interface}"/>
+        <xacro:add_transmission joint_name="r_palm_finger_1_joint" hardware_interface="${hardware_interface}"/>
+        <xacro:add_transmission joint_name="r_palm_finger_2_joint" hardware_interface="${hardware_interface}"/>
+        <xacro:add_transmission joint_name="r_palm_finger_middle_joint" hardware_interface="${hardware_interface}"/>
+    </xacro:macro>
 </robot>

File: victor_description/urdf/robotiq_3finger_gripper.xacro (robot description, xacro)
@@ -1,81 +1,13 @@
 <?xml version="1.0"?>
 <robot xmlns:xacro="http://www.ros.org/wiki/xacro">
-    <xacro:include filename="$(find victor_description)/urdf/robotiq_finger.xacro"/>
-    <xacro:include filename="$(find victor_description)/urdf/robotiq_3finger_gripper.transmission.xacro"/>
-    <xacro:macro name="robotiq_3finger" params="parent prefix hardware_interface *origin">
-        <xacro:property name="joint_damping" value="0.05"/>
-        <joint name="${prefix}_palm_joint" type="fixed">
+    <xacro:macro name="robotiq_3finger" params="prefix side parent *origin hardware_interface">
+        <xacro:include filename="$(find robotiq_3f_gripper_visualization)/cfg/robotiq_hand_macro.urdf.xacro"/>
+        <xacro:robotiq_hand prefix="${prefix}" parent="${parent}">
             <xacro:insert_block name="origin"/>
-            <parent link="${parent}"/>
-            <child link="${prefix}_palm"/>
-        </joint>
-        <link name="${prefix}_palm">
-            <inertial>
-                <origin xyz="0 0 0" rpy="0 0 0"/>
-                <mass value="1"/>
-                <inertia ixx="0.01" ixy="0" ixz="0" iyy="0.01" iyz="0" izz="0.01"/>
-            </inertial>
-            <visual>
-                <origin xyz="0 0 0" rpy="0 0 0"/>
-                <geometry>
-                    <mesh filename="package://victor_description/meshes/robotiq_3finger/palm_visual.stl"/>
-                </geometry>
-                <material name="DarkGray"/>
-            </visual>
-            <collision>
-                <origin xyz="0 0 0" rpy="0 0 0"/>
-                <geometry>
-                    <mesh filename="package://victor_description/meshes/robotiq_3finger/palm_collision.stl"/>
-                </geometry>
-                <material name="DarkGray"/>
-            </collision>
-        </link>
-        <!-- Palm surface aligned with the gripper axis -->
-        <joint name="${prefix}_palm_surface_joint" type="fixed">
-            <parent link="${prefix}_palm"/>
-            <child link="${prefix}_palm_surface"/>
-            <origin xyz="0 0 0.092075" rpy="0 0 0"/>
-        </joint>
-        <link name="${prefix}_palm_surface">
-        </link>
-        <!-- Kuka internal frame has been changed to match our external usage, so identity transform -->
-        <joint name="${prefix}_palm_surface_kuka_joint" type="fixed">
-            <parent link="${prefix}_palm_surface"/>
-            <child link="${prefix}_palm_surface_kuka"/>
-            <origin xyz="0 0 0" rpy="0 0 0"/>
-        </joint>
-        <link name="${prefix}_palm_surface_kuka">
-        </link>
-        <!-- Finger A -->
-        <joint name="${prefix}_fingerA_knuckle" type="fixed">
-            <origin xyz="0.02225040 0 0.06111875" rpy="0 0 0"/>
-            <parent link="${prefix}_palm"/>
-            <child link="${prefix}_fingerA_base"/>
-        </joint>
-        <xacro:robotiq_finger prefix="${prefix}_fingerA" joint_damping="${joint_damping}"/>
-        <!-- Finger B -->
-        <joint name="${prefix}_fingerB_knuckle" type="revolute">
-            <origin xyz="-0.02230120 0.03651250 0.06111875" rpy="0 0 ${PI}"/>
-            <parent link="${prefix}_palm"/>
-            <child link="${prefix}_fingerB_base"/>
-            <axis xyz="-1 0 0"/>
-            <limit lower="${-16 * PI / 180}" upper="${10 * PI / 180}"
-               effort="${max_effort}" velocity="${max_velocity}"/>
-            <dynamics damping="${joint_damping}"/>
-        </joint>
-        <xacro:robotiq_finger prefix="${prefix}_fingerB" joint_damping="${joint_damping}"/>
-        <!-- Finger C -->
-        <joint name="${prefix}_fingerC_knuckle" type="revolute">
-            <origin xyz="-0.02230120 -0.03651250 0.06111875" rpy="0 0 ${PI}"/>
-            <parent link="${prefix}_palm"/>
-            <child link="${prefix}_fingerC_base"/>
-            <axis xyz="1 0 0"/>
-            <limit lower="${-16 * PI / 180}" upper="${10 * PI / 180}"
-               effort="${max_effort}" velocity="${max_velocity}"/>
-            <dynamics damping="${joint_damping}"/>
-        </joint>
-        <xacro:robotiq_finger prefix="${prefix}_fingerC" joint_damping="${joint_damping}"/>
-        <xacro:robotiq_3finger_gripper_transmission hardware_interface="${hardware_interface}"
-                                                    robot_name="${prefix}"/>
+        </xacro:robotiq_hand>
+        <!-- Extensions -->
+        <xacro:include filename="$(find victor_description)/urdf/robotiq_3finger_gripper.gazebo.xacro"/>
+        <xacro:include filename="robotiq_3finger_gripper.transmission.xacro"/>
+        <xacro:robotiq_transmissions hardware_interface="${hardware_interface}"/>
     </xacro:macro>
 </robot>

File: victor_description/urdf/victor.urdf.xacro (robot description, xacro)
@@ -39,19 +39,18 @@
     <xacro:include filename="$(find victor_description)/urdf/iiwa7_to_robotiq_adapter.xacro"/>
     <xacro:iia7_to_robotiq_adapter parent="$(arg robot_name)_left_arm_flange" prefix="$(arg robot_name)_left">
-        <origin xyz="0 0 0" rpy="0 0 0"/>
+        <origin xyz="0 0 -0.01" rpy="0 0 0"/>
     </xacro:iia7_to_robotiq_adapter>
     <xacro:iia7_to_robotiq_adapter parent="$(arg robot_name)_right_arm_flange" prefix="$(arg robot_name)_right">
-        <origin xyz="0 0 0" rpy="0 0 0"/>
+        <origin xyz="0 0 -0.01" rpy="0 0 0"/>
     </xacro:iia7_to_robotiq_adapter>
     <!-- Robotiq grippers -->
-    <!--Import the Robotiq 3 finger macro -->
     <xacro:include filename="$(find victor_description)/urdf/robotiq_3finger_gripper.xacro"/>
-    <xacro:robotiq_3finger parent="$(arg robot_name)_left_gripper_mounting_bracket" prefix="$(arg robot_name)_left_gripper"
+    <xacro:robotiq_3finger parent="$(arg robot_name)_left_gripper_mounting_bracket" prefix="l_" side="left"
                            hardware_interface="$(arg hardware_interface)">
-        <origin xyz="0 0 0.02705" rpy="0 0 ${PI/4}"/> <!-- Offset measured with a tape measure; please confirm/fix this value -->
+        <origin xyz="0 0 0.07" rpy="${PI/2} 0 ${PI/4}"/>
     </xacro:robotiq_3finger>
-    <xacro:robotiq_3finger parent="$(arg robot_name)_right_gripper_mounting_bracket" prefix="$(arg robot_name)_right_gripper"
+    <xacro:robotiq_3finger parent="$(arg robot_name)_right_gripper_mounting_bracket" prefix="r_" side="right"
                            hardware_interface="$(arg hardware_interface)">
-        <origin xyz="0 0 0.02705" rpy="0 0 ${PI/4}"/> <!-- Offset measured with a tape measure; please confirm/fix this value -->
+        <origin xyz="0 0 0.07" rpy="${PI/2} 0 ${PI/4}"/>
     </xacro:robotiq_3finger>
     <!-- Define additional links as "tools", which are useful for planning and getting transforms -->
