Commit message: use position interface, no PID, results in much more stable sim

File: victor_description/urdf/gazebo_utilities.xacro (robot description, xacro)
@@ -99,3 +99,8 @@
         </transmission>
     </xacro:macro>
+    <xacro:macro name="preserve" params="joint_name">
+        <gazebo reference='${joint_name}'>
+            <preserveFixedJoint>true</preserveFixedJoint>
+        </gazebo>
+    </xacro:macro>
 </robot>

File: victor_description/urdf/victor.gazebo.xacro (robot description, xacro)
@@ -1,4 +1,5 @@
 <?xml version="1.0"?>
 <robot xmlns:xacro="http://www.ros.org/wiki/xacro">
+    <xacro:include filename="$(find victor_description)/urdf/gazebo_utilities.xacro"/>
     <gazebo reference="victor_pedestal">
         <visual>
@@ -84,9 +85,5 @@
         <xacro:add_simulation_compliance_arm_helper arm="victor_${side}_arm" index="7"/>
     </xacro:macro>
-    <gazebo reference='right_tool_joint'>
-        <preserveFixedJoint>true</preserveFixedJoint>
-    </gazebo>
-    <gazebo reference='left_tool_joint'>
-        <preserveFixedJoint>true</preserveFixedJoint>
-    </gazebo>
+    <xacro:preserve joint_name="right_tool_joint"/>
+    <xacro:preserve joint_name="left_tool_joint"/>
 </robot>

File: victor_description/urdf/victor.urdf.xacro (robot description, xacro)
@@ -1,6 +1,8 @@
 <?xml version="1.0"?>
 <robot name="victor" xmlns:xacro="http://www.ros.org/wiki/xacro">
+    <xacro:property name="gripper" value="robotiq" />
     <xacro:arg name="robot_name" default="victor"/>
-    <xacro:arg name="hardware_interface" default="hardware_interface/EffortJointInterface"/>
+    <xacro:arg name="hardware_interface" default="hardware_interface/PositionJointInterface"/>
+    <xacro:arg name="gripper_hardware_interface" default="hardware_interface/EffortJointInterface"/>
     <!-- Import Rviz colors -->
     <xacro:include filename="$(find victor_description)/urdf/materials.xacro"/>
@@ -36,22 +38,24 @@
     <link name="$(arg robot_name)_right_arm_world_frame_kuka">
     </link>
-    <!-- arm to gripper adapter -->
-    <xacro:include filename="$(find victor_description)/urdf/iiwa7_to_robotiq_adapter.xacro"/>
-    <xacro:iia7_to_robotiq_adapter parent="$(arg robot_name)_left_arm_flange" prefix="$(arg robot_name)_left">
-        <origin xyz="0 0 -0.01" rpy="0 0 0"/>
-    </xacro:iia7_to_robotiq_adapter>
-    <xacro:iia7_to_robotiq_adapter parent="$(arg robot_name)_right_arm_flange" prefix="$(arg robot_name)_right">
-        <origin xyz="0 0 -0.01" rpy="0 0 0"/>
-    </xacro:iia7_to_robotiq_adapter>
     <!-- Robotiq grippers -->
-    <xacro:include filename="$(find victor_description)/urdf/robotiq_3finger_gripper.xacro"/>
-    <xacro:robotiq_3finger parent="$(arg robot_name)_left_gripper_mounting_bracket" prefix="l_" side="left"
-                           hardware_interface="$(arg hardware_interface)">
-        <origin xyz="0 0 0.07" rpy="${PI/2} 0 ${PI/4}"/>
-    </xacro:robotiq_3finger>
-    <xacro:robotiq_3finger parent="$(arg robot_name)_right_gripper_mounting_bracket" prefix="r_" side="right"
-                           hardware_interface="$(arg hardware_interface)">
-        <origin xyz="0 0 0.07" rpy="${PI/2} 0 ${PI/4}"/>
-    </xacro:robotiq_3finger>
+    <xacro:property name="gripper" value="robotiq">
+        <!-- arm to gripper adapter -->
+        <xacro:include filename="$(find victor_description)/urdf/iiwa7_to_robotiq_adapter.xacro"/>
+        <xacro:iia7_to_robotiq_adapter parent="$(arg robot_name)_left_arm_flange" prefix="$(arg robot_name)_left">
+            <origin xyz="0 0 -0.01" rpy="0 0 0"/>
+        </xacro:iia7_to_robotiq_adapter>
+        <xacro:iia7_to_robotiq_adapter parent="$(arg robot_name)_right_arm_flange" prefix="$(arg robot_name)_right">
+            <origin xyz="0 0 -0.01" rpy="0 0 0"/>
+        </xacro:iia7_to_robotiq_adapter>
+        <xacro:include filename="$(find victor_description)/urdf/robotiq_3finger_gripper.xacro"/>
+        <xacro:robotiq_3finger parent="$(arg robot_name)_left_gripper_mounting_bracket" prefix="l_" side="left"
+                               hardware_interface="$(arg gripper_hardware_interface)">
+            <origin xyz="0 0 0.07" rpy="${PI/2} 0 ${PI/4}"/>
+        </xacro:robotiq_3finger>
+        <xacro:robotiq_3finger parent="$(arg robot_name)_right_gripper_mounting_bracket" prefix="r_" side="right"
+                               hardware_interface="$(arg gripper_hardware_interface)">
+            <origin xyz="0 0 0.07" rpy="${PI/2} 0 ${PI/4}"/>
+        </xacro:robotiq_3finger>
+    </xacro:property>
     <!-- Define additional links as "tools", which are useful for planning and getting transforms -->
     <xacro:include filename="$(find victor_description)/urdf/robotiq_pinch_grasp_tools.xacro"/>
