Commit message: make the hands work
not easily usable though, currently controllable through a position group joint
interface. We need them to respond to GripperCommand

File: victor_description/urdf/robotiq_3finger_gripper.xacro (robot description, xacro)
@@ -61,8 +61,4 @@
             <limit lower="${-16 * PI / 180}" upper="${10 * PI / 180}"
                effort="${max_effort}" velocity="${max_velocity}"/>
-            <safety_controller soft_lower_limit="${-14 * PI / 180}"
-                               soft_upper_limit="${8 * PI / 180}"
-                               k_position="${safety_controller_k_pos}"
-                               k_velocity="${safety_controller_k_vel}"/>
             <dynamics damping="${joint_damping}"/>
         </joint>
@@ -76,8 +72,4 @@
             <limit lower="${-16 * PI / 180}" upper="${10 * PI / 180}"
                effort="${max_effort}" velocity="${max_velocity}"/>
-            <safety_controller soft_lower_limit="${-14 * PI / 180}"
-                               soft_upper_limit="${8 * PI / 180}"
-                               k_position="${safety_controller_k_pos}"
-                               k_velocity="${safety_controller_k_vel}"/>
             <dynamics damping="${joint_damping}"/>
         </joint>

File: victor_description/urdf/robotiq_finger.xacro (robot description, xacro)
@@ -1,6 +1,4 @@
 <?xml version="1.0"?>
 <robot xmlns:xacro="http://www.ros.org/wiki/xacro">
-    <xacro:property name="safety_controller_k_pos" value="0"/>
-    <xacro:property name="safety_controller_k_vel" value="0"/>
     <xacro:property name="joint_damping" value="0.005"/>
     <xacro:property name="max_effort" value="300"/>
@@ -36,8 +34,4 @@
             <limit lower="0" upper="1.2217304763960307"
                    effort="${max_effort}" velocity="${max_velocity}"/>
-            <safety_controller soft_lower_limit="${-35 * PI / 180}"
-                               soft_upper_limit="${35 * PI / 180}"
-                               k_position="${safety_controller_k_pos}"
-                               k_velocity="${safety_controller_k_vel}"/>
             <dynamics damping="${joint_damping}"/>
         </joint>
@@ -71,8 +65,4 @@
             <limit lower="-1" upper="1"
                    effort="${max_effort}" velocity="${max_velocity}"/>
-            <safety_controller soft_lower_limit="${0 * PI / 180}"
-                               soft_upper_limit="${90 * PI / 180}"
-                               k_position="${safety_controller_k_pos}"
-                               k_velocity="${safety_controller_k_vel}"/>
             <dynamics damping="${joint_damping}"/>
         </joint>
@@ -106,8 +96,4 @@
             <limit lower="-1" upper="1"
                    effort="${max_effort}" velocity="${max_velocity}"/>
-            <safety_controller soft_lower_limit="${-25 * PI / 180}"
-                               soft_upper_limit="${73 * PI / 180}"
-                               k_position="${safety_controller_k_pos}"
-                               k_velocity="${safety_controller_k_vel}"/>
             <dynamics damping="${joint_damping}"/>
         </joint>

File: victor_description/urdf/victor.urdf.xacro (robot description, xacro)
@@ -47,8 +47,8 @@
     <!--Import the Robotiq 3 finger macro -->
     <xacro:include filename="$(find victor_description)/urdf/robotiq_3finger_gripper.xacro"/>
-    <xacro:robotiq_3finger parent="$(arg robot_name)_left_gripper_mounting_bracket" prefix="$(arg robot_name)_left_gripper" hardware_interface="hardware_interface/EffortJointInterface">
+    <xacro:robotiq_3finger parent="$(arg robot_name)_left_gripper_mounting_bracket" prefix="$(arg robot_name)_left_gripper" hardware_interface="$(arg hardware_interface)">
         <origin xyz="0 0 0.02705" rpy="0 0 ${PI/4}"/> <!-- Offset measured with a tape measure; please confirm/fix this value -->
     </xacro:robotiq_3finger>
-    <xacro:robotiq_3finger parent="$(arg robot_name)_right_gripper_mounting_bracket" prefix="$(arg robot_name)_right_gripper" hardware_interface="hardware_interface/EffortJointInterface">
+    <xacro:robotiq_3finger parent="$(arg robot_name)_right_gripper_mounting_bracket" prefix="$(arg robot_name)_right_gripper" hardware_interface="$(arg hardware_interface)">
         <origin xyz="0 0 0.02705" rpy="0 0 ${PI/4}"/> <!-- Offset measured with a tape measure; please confirm/fix this value -->
     </xacro:robotiq_3finger>

Commit message: remove fingers because they're getting in the way and closing them is difficult right now

File: victor_description/urdf/robotiq_3finger_gripper.xacro (robot description, xacro)
@@ -31,51 +31,4 @@
             </collision>
         </link>
-        <!-- Palm surface aligned with the gripper axis -->
-        <joint name="${prefix}_palm_surface_joint" type="fixed">
-            <parent link="${prefix}_palm"/>
-            <child link="${prefix}_palm_surface"/>
-            <origin xyz="0 0 0.092075" rpy="0 0 0"/>
-        </joint>
-        <link name="${prefix}_palm_surface">
-        </link>
-        <!-- Kuka internal frame has been changed to match our external usage, so identity transform -->
-        <joint name="${prefix}_palm_surface_kuka_joint" type="fixed">
-            <parent link="${prefix}_palm_surface"/>
-            <child link="${prefix}_palm_surface_kuka"/>
-            <origin xyz="0 0 0" rpy="0 0 0"/>
-        </joint>
-        <link name="${prefix}_palm_surface_kuka">
-        </link>
-        <!-- Finger A -->
-        <joint name="${prefix}_fingerA_knuckle" type="fixed">
-            <origin xyz="0.02225040 0 0.06111875" rpy="0 0 0"/>
-            <parent link="${prefix}_palm"/>
-            <child link="${prefix}_fingerA_base"/>
-        </joint>
-        <xacro:robotiq_finger prefix="${prefix}_fingerA" joint_damping="${joint_damping}"/>
-        <!-- Finger B -->
-        <joint name="${prefix}_fingerB_knuckle" type="revolute">
-            <origin xyz="-0.02230120 0.03651250 0.06111875" rpy="0 0 ${PI}"/>
-            <parent link="${prefix}_palm"/>
-            <child link="${prefix}_fingerB_base"/>
-            <axis xyz="-1 0 0"/>
-            <limit lower="${-16 * PI / 180}" upper="${10 * PI / 180}"
-               effort="${max_effort}" velocity="${max_velocity}"/>
-            <dynamics damping="${joint_damping}"/>
-        </joint>
-        <xacro:robotiq_finger prefix="${prefix}_fingerB" joint_damping="${joint_damping}"/>
-        <!-- Finger C -->
-        <joint name="${prefix}_fingerC_knuckle" type="revolute">
-            <origin xyz="-0.02230120 -0.03651250 0.06111875" rpy="0 0 ${PI}"/>
-            <parent link="${prefix}_palm"/>
-            <child link="${prefix}_fingerC_base"/>
-            <axis xyz="1 0 0"/>
-            <limit lower="${-16 * PI / 180}" upper="${10 * PI / 180}"
-               effort="${max_effort}" velocity="${max_velocity}"/>
-            <dynamics damping="${joint_damping}"/>
-        </joint>
-        <xacro:robotiq_finger prefix="${prefix}_fingerC" joint_damping="${joint_damping}"/>
-        <xacro:robotiq_3finger_gripper_transmission hardware_interface="${hardware_interface}"
-                                                    robot_name="${prefix}"/>
     </xacro:macro>
 </robot>

Commit message: considering supporting two gripper types
but I just figured out why the grippers freaked out before, wrong kp/kd
because it's defined in two places

File: victor_description/urdf/robotiq_3finger_gripper.xacro (robot description, xacro)
@@ -1,13 +1,80 @@
 <?xml version="1.0"?>
 <robot xmlns:xacro="http://www.ros.org/wiki/xacro">
-    <xacro:macro name="robotiq_3finger" params="prefix side parent *origin hardware_interface">
-        <xacro:include filename="$(find robotiq_3f_gripper_visualization)/cfg/robotiq_hand_macro.urdf.xacro"/>
-        <xacro:robotiq_hand prefix="${prefix}" parent="${parent}">
+    <xacro:include filename="$(find victor_description)/urdf/robotiq_finger.xacro"/>
+    <xacro:include filename="$(find victor_description)/urdf/robotiq_3finger_gripper.transmission.xacro"/>
+    <xacro:macro name="robotiq_3finger" params="parent prefix hardware_interface *origin">
+        <joint name="${prefix}_palm_joint" type="fixed">
             <xacro:insert_block name="origin"/>
-        </xacro:robotiq_hand>
-        <!-- Extensions -->
-        <xacro:include filename="$(find victor_description)/urdf/robotiq_3finger_gripper.gazebo.xacro"/>
-        <xacro:include filename="$(find victor_description)/urdf/robotiq_3finger_gripper.transmission.xacro"/>
-        <xacro:robotiq_transmissions prefix="${prefix}" hardware_interface="${hardware_interface}"/>
+            <parent link="${parent}"/>
+            <child link="${prefix}_palm"/>
+        </joint>
+        <link name="${prefix}_palm">
+            <inertial>
+                <origin xyz="0 0 0" rpy="0 0 0"/>
+                <mass value="1"/>
+                <inertia ixx="0.01" ixy="0" ixz="0" iyy="0.01" iyz="0" izz="0.01"/>
+            </inertial>
+            <visual>
+                <origin xyz="0 0 0" rpy="0 0 0"/>
+                <geometry>
+                    <mesh filename="package://victor_description/meshes/robotiq_3finger/palm_visual.stl"/>
+                </geometry>
+                <material name="DarkGray"/>
+            </visual>
+            <collision>
+                <origin xyz="0 0 0" rpy="0 0 0"/>
+                <geometry>
+                    <mesh filename="package://victor_description/meshes/robotiq_3finger/palm_collision.stl"/>
+                </geometry>
+                <material name="DarkGray"/>
+            </collision>
+        </link>
+        <!-- Palm surface aligned with the gripper axis -->
+        <joint name="${prefix}_palm_surface_joint" type="fixed">
+            <parent link="${prefix}_palm"/>
+            <child link="${prefix}_palm_surface"/>
+            <origin xyz="0 0 0.092075" rpy="0 0 0"/>
+        </joint>
+        <link name="${prefix}_palm_surface">
+        </link>
+        <!-- Kuka internal frame has been changed to match our external usage, so identity transform -->
+        <joint name="${prefix}_palm_surface_kuka_joint" type="fixed">
+            <parent link="${prefix}_palm_surface"/>
+            <child link="${prefix}_palm_surface_kuka"/>
+            <origin xyz="0 0 0" rpy="0 0 0"/>
+        </joint>
+        <link name="${prefix}_palm_surface_kuka">
+        </link>
+        <!-- Finger A -->
+        <joint name="${prefix}_fingerA_knuckle" type="fixed">
+            <origin xyz="0.02225040 0 0.06111875" rpy="0 0 0"/>
+            <parent link="${prefix}_palm"/>
+            <child link="${prefix}_fingerA_base"/>
+        </joint>
+        <xacro:robotiq_finger prefix="${prefix}_fingerA"/>
+        <!-- Finger B -->
+        <joint name="${prefix}_fingerB_knuckle" type="revolute">
+            <origin xyz="-0.02230120 0.03651250 0.06111875" rpy="0 0 ${PI}"/>
+            <parent link="${prefix}_palm"/>
+            <child link="${prefix}_fingerB_base"/>
+            <axis xyz="-1 0 0"/>
+            <limit lower="${-16 * PI / 180}" upper="${10 * PI / 180}"
+               effort="${max_effort}" velocity="${max_velocity}"/>
+            <dynamics damping="${joint_damping}"/>
+        </joint>
+        <xacro:robotiq_finger prefix="${prefix}_fingerB"/>
+        <!-- Finger C -->
+        <joint name="${prefix}_fingerC_knuckle" type="revolute">
+            <origin xyz="-0.02230120 -0.03651250 0.06111875" rpy="0 0 ${PI}"/>
+            <parent link="${prefix}_palm"/>
+            <child link="${prefix}_fingerC_base"/>
+            <axis xyz="1 0 0"/>
+            <limit lower="${-16 * PI / 180}" upper="${10 * PI / 180}"
+               effort="${max_effort}" velocity="${max_velocity}"/>
+            <dynamics damping="${joint_damping}"/>
+        </joint>
+        <xacro:robotiq_finger prefix="${prefix}_fingerC"/>
+        <xacro:robotiq_3finger_gripper_transmission hardware_interface="${hardware_interface}"
+                                                    robot_name="${prefix}"/>
     </xacro:macro>
 </robot>

File: victor_description/urdf/victor.urdf.xacro (robot description, xacro)
@@ -1,5 +1,5 @@
 <?xml version="1.0"?>
 <robot name="victor" xmlns:xacro="http://www.ros.org/wiki/xacro">
-    <xacro:property name="gripper" value="robotiq" />
+    <xacro:property name="gripper" value="robotiq_articulated" />
     <xacro:arg name="robot_name" default="victor"/>
     <xacro:arg name="hardware_interface" default="hardware_interface/PositionJointInterface"/>
@@ -39,23 +39,16 @@
     </link>
     <!-- Robotiq grippers -->
-    <xacro:property name="gripper" value="robotiq">
-        <!-- arm to gripper adapter -->
-        <xacro:include filename="$(find victor_description)/urdf/iiwa7_to_robotiq_adapter.xacro"/>
-        <xacro:iia7_to_robotiq_adapter parent="$(arg robot_name)_left_arm_flange" prefix="$(arg robot_name)_left">
-            <origin xyz="0 0 -0.01" rpy="0 0 0"/>
-        </xacro:iia7_to_robotiq_adapter>
-        <xacro:iia7_to_robotiq_adapter parent="$(arg robot_name)_right_arm_flange" prefix="$(arg robot_name)_right">
-            <origin xyz="0 0 -0.01" rpy="0 0 0"/>
-        </xacro:iia7_to_robotiq_adapter>
+    <xacro:if value="${gripper == 'robotiq_articulated'}">
+        <xacro:include filename="robotiq_grippers_articulated.xacro"/>
+    </xacro:if>
+    <xacro:if value="${gripper == 'robotiq'}">
         <xacro:include filename="$(find victor_description)/urdf/robotiq_3finger_gripper.xacro"/>
-        <xacro:robotiq_3finger parent="$(arg robot_name)_left_gripper_mounting_bracket" prefix="l_" side="left"
-                               hardware_interface="$(arg gripper_hardware_interface)">
-            <origin xyz="0 0 0.07" rpy="${PI/2} 0 ${PI/4}"/>
+        <xacro:robotiq_3finger parent="$(arg robot_name)_left_gripper_mounting_bracket" prefix="$(arg robot_name)_left_gripper" hardware_interface="$(arg hardware_interface)">
+            <origin xyz="0 0 0.02705" rpy="0 0 ${PI/4}"/> <!-- Offset measured with a tape measure; please confirm/fix this value -->
         </xacro:robotiq_3finger>
-        <xacro:robotiq_3finger parent="$(arg robot_name)_right_gripper_mounting_bracket" prefix="r_" side="right"
-                               hardware_interface="$(arg gripper_hardware_interface)">
-            <origin xyz="0 0 0.07" rpy="${PI/2} 0 ${PI/4}"/>
+        <xacro:robotiq_3finger parent="$(arg robot_name)_right_gripper_mounting_bracket" prefix="$(arg robot_name)_right_gripper" hardware_interface="$(arg hardware_interface)">
+            <origin xyz="0 0 0.02705" rpy="0 0 ${PI/4}"/> <!-- Offset measured with a tape measure; please confirm/fix this value -->
         </xacro:robotiq_3finger>
-    </xacro:property>
+    </xacro:if>
     <!-- Define additional links as "tools", which are useful for planning and getting transforms -->
     <xacro:include filename="$(find victor_description)/urdf/robotiq_pinch_grasp_tools.xacro"/>
