Commit message: simplifying

File: victor_description/urdf/iiwa.gazebo.xacro (robot description, xacro)
@@ -2,12 +2,4 @@
 <robot xmlns:xacro="http://www.ros.org/wiki/xacro">
   <xacro:macro name="iiwa_gazebo" params="robot_name">
-    <!-- Load Gazebo lib and set the robot namespace -->
-    <!--<xacro:if value="${load_control_plugin}">-->
-      <!--<gazebo>-->
-        <!--<plugin name="gazebo_ros_control" filename="libgazebo_ros_control.so">-->
-          <!--<robotNamespace>/${robot_name}</robotNamespace>-->
-        <!--</plugin>-->
-      <!--</gazebo>-->
-    <!--</xacro:if>-->
     <!-- Link0 -->
     <gazebo reference="${robot_name}_link_0">

File: victor_description/urdf/iiwa7.xacro (robot description, xacro)
@@ -8,7 +8,5 @@
     <xacro:include filename="$(find victor_description)/urdf/utilities.xacro"/>
     <!-- some constants -->
-    <xacro:property name="safety_controller_k_pos" value="100"/>
-    <xacro:property name="safety_controller_k_vel" value="100"/>
-    <xacro:property name="joint_damping" value="0.2"/>
+    <xacro:property name="joint_damping" value="0.5"/>
     <xacro:property name="max_effort" value="300"/>
     <xacro:property name="max_velocity" value="10"/>
@@ -55,8 +53,4 @@
             <limit lower="${-170 * PI / 180}" upper="${170 * PI / 180}"
                    effort="${max_effort}" velocity="${max_velocity}"/>
-            <safety_controller soft_lower_limit="${-168 * PI / 180}"
-                               soft_upper_limit="${168 * PI / 180}"
-                               k_position="${safety_controller_k_pos}"
-                               k_velocity="${safety_controller_k_vel}"/>
             <dynamics damping="${joint_damping}"/>
         </joint>
@@ -89,8 +83,4 @@
             <limit lower="${-120 * PI / 180}" upper="${120 * PI / 180}"
                    effort="${max_effort}" velocity="${max_velocity}"/>
-            <safety_controller soft_lower_limit="${-118 * PI / 180}"
-                               soft_upper_limit="${118 * PI / 180}"
-                               k_position="${safety_controller_k_pos}"
-                               k_velocity="${safety_controller_k_vel}"/>
             <dynamics damping="${joint_damping}"/>
         </joint>
@@ -123,8 +113,4 @@
             <limit lower="${-170 * PI / 180}" upper="${170 * PI / 180}"
                    effort="${max_effort}" velocity="${max_velocity}"/>
-            <safety_controller soft_lower_limit="${-168 * PI / 180}"
-                               soft_upper_limit="${168 * PI / 180}"
-                               k_position="${safety_controller_k_pos}"
-                               k_velocity="${safety_controller_k_vel}"/>
             <dynamics damping="${joint_damping}"/>
         </joint>
@@ -157,8 +143,4 @@
             <limit lower="${-120 * PI / 180}" upper="${120 * PI / 180}"
                    effort="${max_effort}" velocity="${max_velocity}"/>
-            <safety_controller soft_lower_limit="${-118 * PI / 180}"
-                               soft_upper_limit="${118 * PI / 180}"
-                               k_position="${safety_controller_k_pos}"
-                               k_velocity="${safety_controller_k_vel}"/>
             <dynamics damping="${joint_damping}"/>
         </joint>
@@ -191,8 +173,4 @@
             <limit lower="${-170 * PI / 180}" upper="${170 * PI / 180}"
                    effort="${max_effort}" velocity="${max_velocity}"/>
-            <safety_controller soft_lower_limit="${-168 * PI / 180}"
-                               soft_upper_limit="${168 * PI / 180}"
-                               k_position="${safety_controller_k_pos}"
-                               k_velocity="${safety_controller_k_vel}"/>
             <dynamics damping="${joint_damping}"/>
         </joint>
@@ -225,8 +203,4 @@
             <limit lower="${-120 * PI / 180}" upper="${120 * PI / 180}"
                    effort="${max_effort}" velocity="${max_velocity}"/>
-            <safety_controller soft_lower_limit="${-118 * PI / 180}"
-                               soft_upper_limit="${118 * PI / 180}"
-                               k_position="${safety_controller_k_pos}"
-                               k_velocity="${safety_controller_k_vel}"/>
             <dynamics damping="${joint_damping}"/>
         </joint>
@@ -259,8 +233,4 @@
             <limit lower="${-175 * PI / 180}" upper="${175 * PI / 180}"
                    effort="${max_effort}" velocity="${max_velocity}"/>
-            <safety_controller soft_lower_limit="${-173 * PI / 180}"
-                               soft_upper_limit="${173 * PI / 180}"
-                               k_position="${safety_controller_k_pos}"
-                               k_velocity="${safety_controller_k_vel}"/>
             <dynamics damping="${joint_damping}"/>
         </joint>

Commit message: p r e t t y colors

File: victor_description/urdf/iiwa.gazebo.xacro (robot description, xacro)
@@ -1,53 +1,45 @@
 <?xml version="1.0"?>
 <robot xmlns:xacro="http://www.ros.org/wiki/xacro">
-  <xacro:macro name="iiwa_gazebo" params="robot_name">
-    <!-- Link0 -->
-    <gazebo reference="${robot_name}_link_0">
-      <material>Gazebo/Grey</material>
-      <mu1>0.2</mu1>
-      <mu2>0.2</mu2>
-    </gazebo>
-    <!-- Link1 -->
-    <gazebo reference="${robot_name}_link_1">
-      <material>Gazebo/Orange</material>
-      <mu1>0.2</mu1>
-      <mu2>0.2</mu2>
-    </gazebo>
-    <!-- Link2 -->
-    <gazebo reference="${robot_name}_link_2">
-      <material>Gazebo/Orange</material>
-      <mu1>0.2</mu1>
-      <mu2>0.2</mu2>
-    </gazebo>
-    <!-- Link3 -->
-    <gazebo reference="${robot_name}_link_3">
-      <material>Gazebo/Orange</material>
-      <mu1>0.2</mu1>
-      <mu2>0.2</mu2>
-    </gazebo>
-    <!-- Link4 -->
-    <gazebo reference="${robot_name}_link_4">
-      <material>Gazebo/Orange</material>
-      <mu1>0.2</mu1>
-      <mu2>0.2</mu2>
-    </gazebo>
-    <!-- Link5 -->
-    <gazebo reference="${robot_name}_link_5">
-      <material>Gazebo/Orange</material>
-      <mu1>0.2</mu1>
-      <mu2>0.2</mu2>
-    </gazebo>
-    <!-- Link6 -->
-    <gazebo reference="${robot_name}_link_6">
-      <material>Gazebo/Orange</material>
-      <mu1>0.2</mu1>
-      <mu2>0.2</mu2>
-    </gazebo>
-    <!-- Link7 -->
-    <gazebo reference="${robot_name}_link_7">
-      <material>Gazebo/Grey</material>
-      <mu1>0.2</mu1>
-      <mu2>0.2</mu2>
-    </gazebo>
-  </xacro:macro>
+    <xacro:macro name="iiwa_gazebo" params="robot_name">
+        <!-- Link0 -->
+        <gazebo reference="${robot_name}_link_0">
+            <mu1>0.2</mu1>
+            <mu2>0.2</mu2>
+        </gazebo>
+        <!-- Link1 -->
+        <gazebo reference="${robot_name}_link_1">
+            <mu1>0.2</mu1>
+            <mu2>0.2</mu2>
+        </gazebo>
+        <!-- Link2 -->
+        <gazebo reference="${robot_name}_link_2">
+            <mu1>0.2</mu1>
+            <mu2>0.2</mu2>
+        </gazebo>
+        <!-- Link3 -->
+        <gazebo reference="${robot_name}_link_3">
+            <mu1>0.2</mu1>
+            <mu2>0.2</mu2>
+        </gazebo>
+        <!-- Link4 -->
+        <gazebo reference="${robot_name}_link_4">
+            <mu1>0.2</mu1>
+            <mu2>0.2</mu2>
+        </gazebo>
+        <!-- Link5 -->
+        <gazebo reference="${robot_name}_link_5">
+            <mu1>0.2</mu1>
+            <mu2>0.2</mu2>
+        </gazebo>
+        <!-- Link6 -->
+        <gazebo reference="${robot_name}_link_6">
+            <mu1>0.2</mu1>
+            <mu2>0.2</mu2>
+        </gazebo>
+        <!-- Link7 -->
+        <gazebo reference="${robot_name}_link_7">
+            <mu1>0.2</mu1>
+            <mu2>0.2</mu2>
+        </gazebo>
+    </xacro:macro>
 </robot>

File: victor_description/urdf/iiwa7.xacro (robot description, xacro)
@@ -94,5 +94,5 @@
                 <origin xyz="0 0 0" rpy="0 0 0"/>
                 <geometry>
-                    <mesh filename="package://victor_description/meshes/iiwa7/visual/link_2.stl"/>
+                    <mesh filename="package://victor_description/meshes/iiwa7/visual/link_2.dae"/>
                 </geometry>
                 <material name="Orange"/>

File: victor_description/urdf/victor.gazebo.xacro (robot description, xacro)
@@ -1,4 +1,21 @@
 <?xml version="1.0"?>
 <robot xmlns:xacro="http://www.ros.org/wiki/xacro">
+    <gazebo reference="victor_pedestal">
+        <visual>
+            <material>
+                <diffuse>0.2 0.2 0.2 1.0</diffuse>
+                <ambient>0.1 0.1 0.1 1.0</ambient>
+            </material>
+        </visual>
+    </gazebo>
+    <gazebo reference="victor_base_plate">
+        <visual>
+            <material>
+                <diffuse>0.7 0.7 0.7 1.0</diffuse>
+                <ambient>0.3 0.3 0.3 1.0</ambient>
+                <specular>0.9 0.9 0.9 1.0</specular>
+            </material>
+        </visual>
+    </gazebo>
     <gazebo reference="victor_right_arm_link_1">
         <self_collide>1</self_collide>

Commit message: support either fast/robust kinematic grippers, or slow but realistic grippers

File: victor_description/urdf/iiwa.gazebo.xacro (robot description, xacro)
@@ -4,4 +4,5 @@
         <!-- Link0 -->
         <gazebo reference="${robot_name}_link_0">
+            <kinematic>1</kinematic>
             <mu1>0.2</mu1>
             <mu2>0.2</mu2>
@@ -9,4 +10,5 @@
         <!-- Link1 -->
         <gazebo reference="${robot_name}_link_1">
+            <kinematic>1</kinematic>
             <mu1>0.2</mu1>
             <mu2>0.2</mu2>
@@ -14,4 +16,5 @@
         <!-- Link2 -->
         <gazebo reference="${robot_name}_link_2">
+            <kinematic>1</kinematic>
             <mu1>0.2</mu1>
             <mu2>0.2</mu2>
@@ -19,4 +22,5 @@
         <!-- Link3 -->
         <gazebo reference="${robot_name}_link_3">
+            <kinematic>1</kinematic>
             <mu1>0.2</mu1>
             <mu2>0.2</mu2>
@@ -24,4 +28,5 @@
         <!-- Link4 -->
         <gazebo reference="${robot_name}_link_4">
+            <kinematic>1</kinematic>
             <mu1>0.2</mu1>
             <mu2>0.2</mu2>
@@ -29,4 +34,5 @@
         <!-- Link5 -->
         <gazebo reference="${robot_name}_link_5">
+            <kinematic>1</kinematic>
             <mu1>0.2</mu1>
             <mu2>0.2</mu2>
@@ -34,4 +40,5 @@
         <!-- Link6 -->
         <gazebo reference="${robot_name}_link_6">
+            <kinematic>1</kinematic>
             <mu1>0.2</mu1>
             <mu2>0.2</mu2>
@@ -39,4 +46,5 @@
         <!-- Link7 -->
         <gazebo reference="${robot_name}_link_7">
+            <kinematic>1</kinematic>
             <mu1>0.2</mu1>
             <mu2>0.2</mu2>

File: victor_description/urdf/victor.gazebo.xacro (robot description, xacro)
@@ -19,70 +19,4 @@
         </visual>
     </gazebo>
-    <gazebo reference="victor_right_arm_link_1">
-        <self_collide>1</self_collide>
-    </gazebo>
-    <gazebo reference="victor_right_arm_link_2">
-        <self_collide>1</self_collide>
-    </gazebo>
-    <gazebo reference="victor_right_arm_link_3">
-        <self_collide>1</self_collide>
-    </gazebo>
-    <gazebo reference="victor_right_arm_link_4">
-        <self_collide>1</self_collide>
-    </gazebo>
-    <gazebo reference="victor_right_arm_link_5">
-        <self_collide>1</self_collide>
-    </gazebo>
-    <gazebo reference="victor_right_arm_link_6">
-        <self_collide>1</self_collide>
-    </gazebo>
-    <gazebo reference="victor_right_arm_link_7">
-        <self_collide>0</self_collide>
-    </gazebo>
-    <gazebo reference="victor_right_gripper_fingerA_dist">
-        <self_collide>1</self_collide>
-    </gazebo>
-    <gazebo reference="victor_right_gripper_fingerB_dist">
-        <self_collide>1</self_collide>
-    </gazebo>
-    <gazebo reference="victor_right_gripper_fingerC_dist">
-        <self_collide>1</self_collide>
-    </gazebo>
-    <gazebo reference="victor_left_arm_link_1">
-        <self_collide>1</self_collide>
-    </gazebo>
-    <gazebo reference="victor_left_arm_link_2">
-        <self_collide>1</self_collide>
-    </gazebo>
-    <gazebo reference="victor_left_arm_link_3">
-        <self_collide>1</self_collide>
-    </gazebo>
-    <gazebo reference="victor_left_arm_link_4">
-        <self_collide>1</self_collide>
-    </gazebo>
-    <gazebo reference="victor_left_arm_link_5">
-        <self_collide>1</self_collide>
-    </gazebo>
-    <gazebo reference="victor_left_arm_link_6">
-        <self_collide>1</self_collide>
-    </gazebo>
-    <gazebo reference="victor_left_arm_link_7">
-        <self_collide>0</self_collide>
-    </gazebo>
-    <gazebo reference="victor_left_gripper_fingerA_dist">
-        <self_collide>1</self_collide>
-    </gazebo>
-    <gazebo reference="victor_left_gripper_fingerB_dist">
-        <self_collide>1</self_collide>
-    </gazebo>
-    <gazebo reference="victor_left_gripper_fingerC_dist">
-        <self_collide>1</self_collide>
-    </gazebo>
-    <xacro:macro name="add_simulation_compliance" params="side">
-        <xacro:add_simulation_compliance_finger_helper finger="victor_${side}_gripper_fingerA"/>
-        <xacro:add_simulation_compliance_finger_helper finger="victor_${side}_gripper_fingerB"/>
-        <xacro:add_simulation_compliance_finger_helper finger="victor_${side}_gripper_fingerB"/>
-        <xacro:add_simulation_compliance_arm_helper arm="victor_${side}_arm" index="7"/>
-    </xacro:macro>
     <xacro:preserve joint_name="right_tool_joint"/>
     <xacro:preserve joint_name="left_tool_joint"/>

File: victor_description/urdf/victor.urdf.xacro (robot description, xacro)
@@ -1,8 +1,7 @@
 <?xml version="1.0"?>
 <robot name="victor" xmlns:xacro="http://www.ros.org/wiki/xacro">
-    <xacro:property name="gripper" value="robotiq_articulated" />
+    <xacro:property name="gripper" value="robotiq" />
     <xacro:arg name="robot_name" default="victor"/>
     <xacro:arg name="hardware_interface" default="hardware_interface/PositionJointInterface"/>
-    <xacro:arg name="gripper_hardware_interface" default="hardware_interface/EffortJointInterface"/>
     <!-- Import Rviz colors -->
     <xacro:include filename="$(find victor_description)/urdf/materials.xacro"/>
@@ -38,16 +37,18 @@
     <link name="$(arg robot_name)_right_arm_world_frame_kuka">
     </link>
+    <!-- arm to gripper adapter -->
+    <xacro:include filename="$(find victor_description)/urdf/iiwa7_to_robotiq_adapter.xacro"/>
+    <xacro:iia7_to_robotiq_adapter parent="$(arg robot_name)_left_arm_flange" prefix="$(arg robot_name)_left">
+        <origin xyz="0 0 -0.01" rpy="0 0 0"/>
+    </xacro:iia7_to_robotiq_adapter>
+    <xacro:iia7_to_robotiq_adapter parent="$(arg robot_name)_right_arm_flange" prefix="$(arg robot_name)_right">
+        <origin xyz="0 0 -0.01" rpy="0 0 0"/>
+    </xacro:iia7_to_robotiq_adapter>
     <!-- Robotiq grippers -->
-    <xacro:if value="${gripper == 'robotiq_articulated'}">
-        <xacro:include filename="$(find victor_description)/urdf/robotiq_grippers_articulated.xacro"/>
+    <xacro:if value="${gripper == 'kinematic_robotiq'}">
+        <xacro:include filename="$(find victor_description)/urdf/kinematic_robotiq_grippers.xacro"/>
     </xacro:if>
     <xacro:if value="${gripper == 'robotiq'}">
-        <xacro:include filename="$(find victor_description)/urdf/robotiq_3finger_gripper.xacro"/>
-        <xacro:robotiq_3finger parent="$(arg robot_name)_left_gripper_mounting_bracket" prefix="$(arg robot_name)_left_gripper" hardware_interface="$(arg gripper_hardware_interface)">
-            <origin xyz="0 0 0.02705" rpy="0 0 ${PI/4}"/> <!-- Offset measured with a tape measure; please confirm/fix this value -->
-        </xacro:robotiq_3finger>
-        <xacro:robotiq_3finger parent="$(arg robot_name)_right_gripper_mounting_bracket" prefix="$(arg robot_name)_right_gripper" hardware_interface="$(arg gripper_hardware_interface)">
-            <origin xyz="0 0 0.02705" rpy="0 0 ${PI/4}"/> <!-- Offset measured with a tape measure; please confirm/fix this value -->
-        </xacro:robotiq_3finger>
+        <xacro:include filename="$(find victor_description)/urdf/robotiq_grippers.xacro"/>
     </xacro:if>
     <!-- Define additional links as "tools", which are useful for planning and getting transforms -->
@@ -60,6 +61,4 @@
     <xacro:add_gazebo_control_plugin robot_namespace="$(arg robot_name)"/>
     <xacro:add_moveit_planning_scene_plugin robot_namespace="$(arg robot_name)" root_frame_id="victor_root"/>
-    <xacro:add_simulation_compliance side="left"/>
-    <xacro:add_simulation_compliance side="right"/>
     <!-- Rigidly attach Victor to the Gazebo world -->
     <xacro:add_gazebo_fixed_link base_link="$(arg robot_name)_root"/>
