Commit message: Added collision geometry to account for the rope attachments to URDF and SRDF.

File: victor_description/urdf/victor.urdf.xacro (robot description, xacro)
@@ -53,4 +53,42 @@
         <origin xyz="0 0 0.02705" rpy="0 0 ${PI/4}"/> <!-- Offset measured with a tape measure; please confirm/fix this value -->
     </xacro:robotiq_3finger>
+    <link name="$(arg robot_name)_left_tool_placeholder">
+        <visual>
+            <origin xyz="0 0 0" rpy="0 0 0"/>
+            <geometry>
+                <cylinder length="${6 * 0.0254}" radius="0.03"/>
+            </geometry>
+        </visual>
+        <collision>
+            <origin xyz="0 0 0" rpy="0 0 0"/>
+            <geometry>
+                <cylinder length="${6 * 0.0254}" radius="0.03"/>
+            </geometry>
+        </collision>
+    </link>
+    <joint name="$(arg robot_name)_left_tool_joint" type="fixed">
+        <parent link="$(arg robot_name)_left_gripper_palm_surface"/>
+        <child link="$(arg robot_name)_left_tool_placeholder"/>
+        <origin xyz="0 0 ${3 * 0.0254}"/>
+    </joint>
+    <link name="$(arg robot_name)_right_tool_placeholder">
+        <visual>
+            <origin xyz="0 0 0" rpy="0 0 0"/>
+            <geometry>
+                <cylinder length="${6 * 0.0254}" radius="0.03"/>
+            </geometry>
+        </visual>
+        <collision>
+            <origin xyz="0 0 0" rpy="0 0 0"/>
+            <geometry>
+                <cylinder length="${6 * 0.0254}" radius="0.03"/>
+            </geometry>
+        </collision>
+    </link>
+    <joint name="$(arg robot_name)_right_tool_joint" type="fixed">
+        <parent link="$(arg robot_name)_right_gripper_palm_surface"/>
+        <child link="$(arg robot_name)_right_tool_placeholder"/>
+        <origin xyz="0 0 ${3 * 0.0254}"/>
+    </joint>
     <!-- Add Gazebo properties for whole robot -->
     <xacro:include filename="$(find victor_description)/urdf/gazebo_utilities.xacro"/>

Commit message: remove unused stuff from srdf
technically we need two srdfs for the different grippers, but no one is
using the other gripper rn

File: victor_description/urdf/victor.urdf.xacro (robot description, xacro)
@@ -1,5 +1,5 @@
 <?xml version="1.0"?>
 <robot name="victor" xmlns:xacro="http://www.ros.org/wiki/xacro">
-    <xacro:property name="gripper" value="robotiq" />
+    <xacro:property name="gripper" value="kinematic_robotiq" />
     <xacro:arg name="robot_name" default="victor"/>
     <xacro:arg name="hardware_interface" default="hardware_interface/PositionJointInterface"/>
